File: BILLEE_Rover_Control_Module_V1/inputs_estop.kicad_sch (KiCad schematic)
At the start: 0 parts

Commit message: Updated Doc with new I2C Device and added ESTOP subsystem to Schematic
Parts:
- added CN1: LOGIC_PWR_XT60, PDB_LCSC:CONN-TH_XT60PW-M, symbol PDB_LSCS_Libs:XT60PW-M
- added SW1: ESTOP, Button_Switch_SMD:Nidec_Copal_CAS-120A, symbol Switch:SW_Nidec_CAS-120A1
- added U1, U2, U3: SN74LVC08APWR, PDB_LCSC:TSSOP-14_L5.0-W4.4-P0.65-LS6.4-BL, symbol PDB_LSCS_Libs:SN74LVC08APWR
- added U4: Screw Terminal, PDB_LCSC:CONN-TH_P5.00_KF301-5.0-2P, symbol PDB_LSCS_Libs:KF301-5.0-2P
Connections:
- new net: SW1.2 (B), U4.1
- new net +22.2V_LOGIC: CN1.2 (+)
- new net +3.3V_RP2350_VCC: SW1.3 (A), U1.14 (VCC), U2.14 (VCC), U3.14 (VCC)
- new net BUFF_ARM_EN: U2.10 (3B)
- new net BUFF_AUX_22.2V: U3.2 (1B)
- new net BUFF_DRIVE_EN_1: U1.2 (1B)
- new net BUFF_DRIVE_EN_2: U1.5 (2B)
- new net BUFF_DRIVE_EN_3: U1.10 (3B)
- new net BUFF_DRIVE_EN_4: U1.13 (4B)
- new net BUFF_DRIVE_EN_5: U2.2 (1B)
- new net BUFF_DRIVE_EN_6: U2.5 (2B)
- new net BUFF_E_STOP_STATUS: U1.1 (1A), U1.12 (4A), U1.4 (2A), U1.9 (3A), U2.1 (1A), U2.12 (4A), U2.4 (2A), U2.9 (3A), U3.1 (1A), U3.4 (2A), U4.2
- new net BUFF_SCIENCE_EN: U2.13 (4B)
- new net GND: CN1.1 (-), CN1.3, CN1.4, SW1.1 (C), U1.7 (GND), U2.7 (GND), U3.7 (GND)
- no-connect marks 0 -> 8
Other:
- note added: "ESTOP / Power Circuit"
