File: BILLEE_Rover_Control_Module_V1/untitled.kicad_sch (KiCad schematic)
At the start: 39 parts, among them J1 USB_B_Micro, J2 Conn_02x18_Odd_Even, J3 Conn_02x18_Odd_Even, J4 SM03B-SRSS-TB, SW2 SW_Push, SW3 SW_Push, U15 W25Q128JVS, U16 NCP1117-3.3_SOT223, U17 RP2350_60QFN, Y1 ABM8-272-T3

Commit message: Lots of Goodies. Getting the ball rolling
Merged Jasons changed on starting the RP2350.
I refactored his symbols, fixed some connections, and started implementing the buffers as well as all the necessary GPIO connections.
Parts:
- removed C15, C16, C17, C18, C19: 100n, Capacitor_SMD:C_0402_1005Metric, symbol Device:C
- removed C20: 10u, Capacitor_SMD:C_0805_2012Metric, symbol Device:C
- removed J1: USB_B_Micro, Connector_USB:USB_Micro-B_Amphenol_10103594-0001LF_Horizontal, symbol Connector:USB_B_Micro
- removed J2, J3: Conn_02x18_Odd_Even, Connector_PinHeader_2.54mm:PinHeader_2x18_P2.54mm_Vertical, symbol Connector_Generic:Conn_02x18_Odd_Even
- removed J4: SM03B-SRSS-TB, Connector_JST:JST_SH_SM03B-SRSS-TB_1x03-1MP_P1.00mm_Horizontal, symbol Connector_Generic_MountingPin:Conn_01x03_MountingPin
- removed R1, R9: DNF, Resistor_SMD:R_0402_1005Metric, symbol Device:R
- removed R10: 0, Resistor_SMD:R_0402_1005Metric, symbol Device:R
- removed R2, R4, R6: 1k, Resistor_SMD:R_0402_1005Metric, symbol Device:R
- removed R5: 33, Resistor_SMD:R_0402_1005Metric, symbol Device:R
- removed R7, R8: 27, Resistor_SMD:R_0402_1005Metric, symbol Device:R
- removed U15: W25Q128JVS, Package_SO:SOIC-8_5.23x5.23mm_P1.27mm, symbol Memory_Flash:W25Q128JVS
- removed U16: NCP1117-3.3_SOT223, Package_TO_SOT_SMD:SOT-223-3_TabPin2, symbol Regulator_Linear:NCP1117-3.3_SOT223
- removed U17: RP2350_60QFN, RP2350_60QFN_minimal:RP2350-QFN-60-1EP_7x7_P0.4mm_EP3.4x3.4mm_ThermalVias, symbol MCU_RaspberryPi_RP2350:RP2350_60QFN
- removed Y1: ABM8-272-T3, Crystal:Crystal_SMD_3225-4Pin_3.2x2.5mm, symbol Device:Crystal_GND24
- added D1: PWR_LED, symbol Device:LED
- added J1: 2.54mm Header, Connector_PinHeader_2.54mm:PinHeader_1x03_P2.54mm_Vertical, symbol Connector:Conn_01x03_Socket
- added R1: DNF, Resistor_SMD:R_0402_1005Metric, symbol Device:R_US
- added R10, R9: 5.1k, EPS:R0402, symbol Device:R_US
- added R11, R6: 1k, Resistor_SMD:R_0402_1005Metric, symbol Device:R_US
- added R12, R13, R14, R15, R16, R17, R18, R19, R20, R21, R22, R23: 10k, symbol Device:R_US
- added R2: 0, Resistor_SMD:R_0402_1005Metric, symbol Device:R_US
- added R24, R3, R4: 10k, Resistor_SMD:R_0402_1005Metric, symbol Device:R_US
- added R25: 2k, symbol Device:R_US
- added R5: 33, Resistor_SMD:R_0402_1005Metric, symbol Device:R_US
- added R7, R8: 27, Resistor_SMD:R_0402_1005Metric, symbol Device:R_US
- added U15: W25Q128JVS, PDB_LCSC:SOIC-8_L5.3-W5.3-P1.27-LS8.0-BL, symbol PDB_LSCS_Libs:W25Q128JVSIQTR
- added U16: RP2350A_C42411118, PDB_LCSC:QFN-60_L7.0-W7.0-P0.40-TL-EP3.4, symbol PDB_LCSC:RP2350A_C42411118
- added U17, U18: TCA4307DGKR, PDB_LCSC:VSSOP-8_L3.0-W3.0-P0.65-LS4.9-BL, symbol PDB_LSCS_Libs:TCA4307DGKR
- added U19, U20: SN74LVC244APWR, PDB_LCSC:TSSOP-20_L6.5-W4.4-P0.65-LS6.4-BL, symbol PDB_LSCS_Libs:SN74LVC244APWR
- added USB1: TYPE-C 16PIN 2MD, PDB_LCSC:USB-C-SMD_TYPE-C-16PIN-2MD-073, symbol PDB_LSCS_Libs:TYPE-C16PIN2MD
- added Y1: ABM8_262_T3, PDB_LCSC:CRYSTAL-SMD_4P-L3.2-W2.5-BL, symbol PDB_LSCS_Libs:ABM8-272-T3_C20625731
- C10, C11: value 4.7u -> 100n
- C13, C14: value 100n -> 15p; LCSC Part (none) -> C86285
- C2: value 10u -> 4.7u; footprint Capacitor_SMD:C_0805_2012Metric -> Capacitor_SMD:C_0603_1608Metric
- C3: value 15p -> 4.7u; footprint Capacitor_SMD:C_0402_1005Metric -> Capacitor_SMD:C_0603_1608Metric
- C4: value 15p -> 100n
- C5: value 100n -> 4.7u
- C6: value 10u -> 100n; footprint Capacitor_SMD:C_0805_2012Metric -> Capacitor_SMD:C_0402_1005Metric
- C7, C8: value 4.7u -> 100n; footprint RP2350_60QFN_minimal:C_0402_1005Metric_small_pads -> Capacitor_SMD:C_0402_1005Metric
- L1: footprint RP2350_60QFN_minimal:L_pol_2016 -> (none); LCSC Part (none) -> C42411119
- SW2: value SW_Push -> KMR2; footprint Button_Switch_SMD:SW_Push_1P1T_NO_Vertical_Wuerth_434133025816 -> Button_Switch_SMD:SW_Push_1P1T_NO_CK_KMR2
- SW3: value SW_Push -> RESET SW; footprint Button_Switch_SMD:SW_Push_1P1T_NO_Vertical_Wuerth_434133025816 -> Button_Switch_SMD:SW_Push_1P1T_NO_CK_KMR2
Connections:
- net VBUS is gone; now on net +3.3V_RP2350_VCC: C2.1
- net +1V1: now also C3.1, U16.50 (VREG_FB); no longer C11.1, C12.1, C8.1, C9.1
- net FLASH_SS: now also R1.2, R2.2, R4.2, U15.1 (~{CS})
- net GND: now also C13.1, C14.1, D1.1 (K), J1.1 (Pin_1), R10.2, R3.1, R9.2, U15.4 (GND), U16.47 (VREG_PGND), U16.61 (GND), U17.4 (GND), U18.4 (GND), U19.1 (~{1OE}), U19.10 (GND), U19.19 (~{2OE}), U20.1 (~{1OE}), U20.10 (GND), U20.19 (~{2OE}), USB1.1 (GND), USB1.12 (GND), USB1.13 (SHELL), USB1.14 (SHELL), Y1.2, Y1.4; no longer C13.2, C14.2
- net QSPI_SCLK: now also U15.6 (CLK), U16.56 (QSPI_SCLK)
- net QSPI_SD0: now also U15.5 (DI(IO0)), U16.57 (QSPI_SD0)
- net QSPI_SD1: now also U15.2 (DO(IO1)), U16.59 (QSPI_SD1)
- net QSPI_SD2: now also U15.3 (IO2), U16.58 (QSPI_SD2)
- net QSPI_SD3: now also U15.7 (IO3), U16.55 (QSPI_SD3)
- net QSPI_SS: now also R2.1, R6.2, U16.60 (QSPI_SS)
- net RUN: now also U16.26 (RUN)
- net SWCLK: now also J1.2 (Pin_2), U16.24 (SWCLK)
- net SWD: now also J1.3 (Pin_3), U16.25 (SWD)
- net USB_D+: now also R7.2, USB1.6 (DP1), USB1.8 (DP2)
- net USB_D-: now also R8.2, USB1.5 (DN2), USB1.7 (DN1)
- net VREG_AVDD: now also C5.1, R5.2, U16.46 (VREG_AVDD); no longer C10.1
- net VREG_LX: now also U16.48 (VREG_LX)
- net XIN: now also C13.2, U16.21 (XIN), Y1.1; no longer C3.1
- net XOUT: now also R11.2, U16.22 (XOUT)
- net ~{USB_BOOT}: now also R6.1
- net SW_RUN_R: now reaches SW3.1
- net SW_RUN_R: now also R3.2
- net +3.3V_RP2350_VCC: now reaches C4.1
- net +3.3V_RP2350_VCC: now also C10.1, C11.1, C12.1, C6.1, C7.1, C8.1, C9.1, R12.2, R13.2, R14.2, R15.2, R16.2, R17.2, R18.2, R19.2, R20.2, R21.2, R22.2, R23.2, R25.1, R4.1, R5.1, U15.8 (VCC), U16.1 (IOVDD), U16.11 (IOVDD), U16.20 (IOVDD), U16.30 (IOVDD), U16.38 (IOVDD), U16.44 (ADC_AVDD), U16.45 (IOVDD), U16.49 (VREG_VIN), U16.53 (USB_OTP_VDD), U16.54 (QSPI_IOVDD), U17.8 (VCC), U18.8 (VCC), U19.20 (VCC), U20.20 (VCC)
- removed net +3V3: C13.1, C14.1, C5.1, C6.1, C7.1
- new net: R9.1, USB1.4 (CC1)
- new net: R24.1, U16.17 (GPIO13)
- new net: R10.1, USB1.10 (CC2)
- new net: D1.2 (A), R25.2
- new net: R17.1, U17.5 (READY)
- new net: R13.1, U17.1 (EN)
- new net: R20.1, U18.1 (EN)
- new net: R23.1, U18.5 (READY)
- new net BUFF_ARM_EN: U19.5 (2Y3)
- new net BUFF_AUX_22.2V: U20.18 (1Y1)
- new net BUFF_DRIVE_EN_1: U19.18 (1Y1)
- new net BUFF_DRIVE_EN_2: U19.16 (1Y2)
- new net BUFF_DRIVE_EN_3: U19.14 (1Y3)
- new net BUFF_DRIVE_EN_4: U19.12 (1Y4)
- new net BUFF_DRIVE_EN_5: U19.9 (2Y1)
- new net BUFF_DRIVE_EN_6: U19.7 (2Y2)
- new net BUFF_E_STOP_STATUS: R24.2
- new net BUFF_SCIENCE_EN: U19.3 (2Y4)
- new net BUFF_SCL_0: R15.1, U17.2 (SCLOUT)
- new net BUFF_SCL_1: R21.1, U18.2 (SCLOUT)
- new net BUFF_SDA_0: R16.1, U17.7 (SDAOUT)
- new net BUFF_SDA_1: R22.1, U18.7 (SDAOUT)
- new net DP_D+: R7.1, U16.52 (USB_DP)
- new net DP_D-: R8.1, U16.51 (USB_DM)
- new net GPIO_AUX_22.2V: U16.16 (GPIO12), U20.2 (1A1)
- new net GPIO_DRIVE_EN_1: U16.7 (GPIO4), U19.2 (1A1)
- new net GPIO_DRIVE_EN_2: U16.8 (GPIO5), U19.4 (1A2)
- new net GPIO_DRIVE_EN_3: U16.9 (GPIO6), U19.6 (1A3)
- new net GPIO_DRIVE_EN_4: U16.10 (GPIO7), U19.8 (1A4)
- new net GPIO_DRIVE_EN_5: U16.12 (GPIO8), U19.11 (2A1)
- new net GPIO_DRIVE_EN_6: U16.13 (GPIO9), U19.13 (2A2)
- new net GPIO_SCIENCE_EN: U16.15 (GPIO11), U19.17 (2A4)
- new net GPIO__ARM_EN: U16.14 (GPIO10), U19.15 (2A3)
- new net PI_SCL_0: R12.1, U16.3 (GPIO1), U17.3 (SCLIN)
- new net PI_SCL_1: R19.1, U16.5 (GPIO3), U18.3 (SCLIN)
- new net PI_SDA_0: R14.1, U16.2 (GPIO0), U17.6 (SDAIN)
- new net PI_SDA_1: R18.1, U16.4 (GPIO2), U18.6 (SDAIN)
- new net VBUS_USB: USB1.11 (VBUS), USB1.2 (VBUS)
- new net XOUT_R: C14.2, R11.1, Y1.3
- no-connect marks 1 -> 33
Other:
- note added: "1V1 Integrated VReg @ 200mA"
- note added: "90 0hm Differential Pairs"
- note added: "Crystal"
- note added: "Debug"
- note added: "I2C/GPIO Buffers"
- note added: "I2C0 Buffer"
- note added: "I2C1 Buffer"
- note added: "Make Resistors as close as possible to the RP2350."
- note added: "Make sure PCB trace is short"
- note added: "RP2350A MPU"
- note added: "USB-C"
- note removed: "12MHz Crystal"
- note removed: "IOs"
- note removed: "JST Debug Connector"
- note removed: "Make sure R7 and R8 are close to RP2350"
- note removed: "Power"

Commit message: Implemented Logic Subsystem
Implemented all of the Logic subsystem, missing reverse circuit protection.
Parts:
- removed U15: W25Q128JVS, PDB_LCSC:SOIC-8_L5.3-W5.3-P1.27-LS8.0-BL, symbol PDB_LSCS_Libs:W25Q128JVSIQTR
- removed U16: RP2350A_C42411118, PDB_LCSC:QFN-60_L7.0-W7.0-P0.40-TL-EP3.4, symbol PDB_LCSC:RP2350A_C42411118
- removed U17, U18: TCA4307DGKR, PDB_LCSC:VSSOP-8_L3.0-W3.0-P0.65-LS4.9-BL, symbol PDB_LSCS_Libs:TCA4307DGKR
- removed U19, U20: SN74LVC244APWR, PDB_LCSC:TSSOP-20_L6.5-W4.4-P0.65-LS6.4-BL, symbol PDB_LSCS_Libs:SN74LVC244APWR
- removed USB1: TYPE-C 16PIN 2MD, PDB_LCSC:USB-C-SMD_TYPE-C-16PIN-2MD-073, symbol PDB_LSCS_Libs:TYPE-C16PIN2MD
- removed Y1: ABM8_262_T3, PDB_LCSC:CRYSTAL-SMD_4P-L3.2-W2.5-BL, symbol PDB_LSCS_Libs:ABM8-272-T3_C20625731
- added U15: W25Q128JVSIQTR, PDB_LCSC:SOIC-8_L5.3-W5.3-P1.27-LS8.0-BL, symbol PDB_LCSC_Libs:W25Q128JVSIQTR
- added U16, U19: SN74LVC244APWR, PDB_LCSC:TSSOP-20_L6.5-W4.4-P0.65-LS6.4-BL, symbol PDB_LCSC_Libs:SN74LVC244APWR
- added U17: ABM8-272-T3_C20625731, PDB_LCSC:CRYSTAL-SMD_4P-L3.2-W2.5-BL, symbol PDB_LCSC_Libs:ABM8-272-T3_C20625731
- added U18: RP2350A_C42411118, PDB_LCSC:QFN-60_L7.0-W7.0-P0.40-TL-EP3.4, symbol PDB_LCSC_Libs:RP2350A_C42411118
- added U21, U22: TCA4307DGKR, PDB_LCSC:VSSOP-8_L3.0-W3.0-P0.65-LS4.9-BL, symbol PDB_LCSC_Libs:TCA4307DGKR
- added USB1: TYPE-C 16PIN 2MD, PDB_LCSC:USB-C-SMD_TYPE-C-16PIN-2MD-073, symbol PDB_LCSC_Libs:TYPE-C16PIN2MD
Connections:
- net +1V1: now also U18.50 (VREG_FB)
- net +3.3V_RP2350_VCC: now also U15.8 (VCC), U16.20 (VCC), U18.1 (IOVDD), U18.11 (IOVDD), U18.20 (IOVDD), U18.30 (IOVDD), U18.38 (IOVDD), U18.44 (ADC_AVDD), U18.45 (IOVDD), U18.49 (VREG_VIN), U18.53 (USB_OTP_VDD), U18.54 (QSPI_IOVDD), U19.20 (VCC), U21.8 (VCC), U22.8 (VCC)
- net BUFF_ARM_EN: now also U16.5 (2Y3)
- net BUFF_AUX_22.2V: now also U19.18 (1Y1)
- net BUFF_DRIVE_EN_1: now also U16.18 (1Y1)
- net BUFF_DRIVE_EN_2: now also U16.16 (1Y2)
- net BUFF_DRIVE_EN_3: now also U16.14 (1Y3)
- net BUFF_DRIVE_EN_4: now also U16.12 (1Y4)
- net BUFF_DRIVE_EN_5: now also U16.9 (2Y1)
- net BUFF_DRIVE_EN_6: now also U16.7 (2Y2)
- net BUFF_SCIENCE_EN: now also U16.3 (2Y4)
- net BUFF_SCL_0: now also U21.2 (SCLOUT)
- net BUFF_SCL_1: now also U22.2 (SCLOUT)
- net BUFF_SDA_0: now also U21.7 (SDAOUT)
- net BUFF_SDA_1: now also U22.7 (SDAOUT)
- net DP_D+: now also U18.52 (USB_DP)
- net DP_D-: now also U18.51 (USB_DM)
- net FLASH_SS: now also U15.1 (~{CS})
- net GND: now also U15.4 (GND), U16.1 (~{1OE}), U16.10 (GND), U16.19 (~{2OE}), U17.2, U17.4, U18.47 (VREG_PGND), U18.61 (GND), U19.1 (~{1OE}), U19.10 (GND), U19.19 (~{2OE}), U21.4 (GND), U22.4 (GND), USB1.1 (GND), USB1.12 (GND), USB1.13 (SHELL), USB1.14 (SHELL)
- net GPIO_AUX_22.2V: now also U18.16 (GPIO12), U19.2 (1A1)
- net GPIO_DRIVE_EN_1: now also U16.2 (1A1), U18.7 (GPIO4)
- net GPIO_DRIVE_EN_2: now also U16.4 (1A2), U18.8 (GPIO5)
- net GPIO_DRIVE_EN_3: now also U16.6 (1A3), U18.9 (GPIO6)
- net GPIO_DRIVE_EN_4: now also U16.8 (1A4), U18.10 (GPIO7)
- net GPIO_DRIVE_EN_5: now also U16.11 (2A1), U18.12 (GPIO8)
- net GPIO_DRIVE_EN_6: now also U16.13 (2A2), U18.13 (GPIO9)
- net GPIO_SCIENCE_EN: now also U16.17 (2A4), U18.15 (GPIO11)
- net GPIO__ARM_EN: now also U16.15 (2A3), U18.14 (GPIO10)
- net PI_SCL_0: now also U18.3 (GPIO1), U21.3 (SCLIN)
- net PI_SCL_1: now also U18.5 (GPIO3), U22.3 (SCLIN)
- net PI_SDA_0: now also U18.2 (GPIO0), U21.6 (SDAIN)
- net PI_SDA_1: now also U18.4 (GPIO2), U22.6 (SDAIN)
- net QSPI_SCLK: now also U15.6 (CLK), U18.56 (QSPI_SCLK)
- net QSPI_SD0: now also U15.5 (DI(IO0)), U18.57 (QSPI_SD0)
- net QSPI_SD1: now also U15.2 (DO(IO1)), U18.59 (QSPI_SD1)
- net QSPI_SD2: now also U15.3 (IO2), U18.58 (QSPI_SD2)
- net QSPI_SD3: now also U15.7 (IO3), U18.55 (QSPI_SD3)
- net QSPI_SS: now also U18.60 (QSPI_SS)
- net RUN: now also U18.26 (RUN)
- net SWCLK: now also U18.24 (SWCLK)
- net SWD: now also U18.25 (SWD)
- net USB_D+: now also USB1.6 (DP1), USB1.8 (DP2)
- net USB_D-: now also USB1.5 (DN2), USB1.7 (DN1)
- net VBUS_USB: now also USB1.11 (VBUS), USB1.2 (VBUS)
- net VREG_AVDD: now also U18.46 (VREG_AVDD)
- net VREG_LX: now also U18.48 (VREG_LX)
- net XIN: now also U17.1, U18.21 (XIN)
- net XOUT: now also U18.22 (XOUT)
- net XOUT_R: now also U17.3
- net at R9.1: now also USB1.4 (CC1)
- net at R24.1: now also U18.17 (GPIO13)
- net at R10.1: now also USB1.10 (CC2)
- net at R17.1: now also U21.5 (READY)
- net at R13.1: now also U21.1 (EN)
- net at R20.1: now also U22.1 (EN)
- net at R23.1: now also U22.5 (READY)
