File: BILLEE_Rover_Control_Module_V1/gate driver + mosfet.kicad_sch (KiCad schematic)
At the start: 10 parts, among them Q1 IPT007N06N, U12 LTC7001IMSE#PBF

Commit message: WIP Checkpoint
Parts:
- removed C45: 47uF, symbol Device:C
- removed C46, C47: 0.47uF, symbol Device:C
- removed C48: 15mF, symbol Device:C
- removed Q1: IPT007N06N, PDB_LCSC:HSOF-8_IPT007N06N, symbol PDB_LCSC_Libs:IPT007N06N
- removed R24: 590K, symbol Device:R_US
- removed R60: 12.1K, symbol Device:R_US
- removed R70: 220k, symbol Device:R_US
- removed R71: 10, symbol Device:R_US
- removed U12: LTC7001IMSE#PBF, PDB_LCSC:MSOP-10_L3.0-W3.0-P0.50-LS4.9-BL-EP, symbol PDB_LCSC_Libs:LTC7001IMSE#PBF
