File: BILLEE_Rover_Control_Module_V1/BILLEE_Rover_Control_Module_V1.kicad_sch (KiCad schematic)
At the start: 0 parts

Commit message: sw
Other:
- note added: "Ubiquiti Horn"
Changed lines of the file:
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@@
 	(rectangle
 		(start 278.13 101.6)
-		(end 297.815 179.705)
+		(end 297.815 182.245)
 		(stroke
 			(width 0)
@@
 		(effects
 			(font
+				(size 1.27 1.27)
+			)
+		)
+	)
+	(text "Ubiquiti Horn"
+		(exclude_from_sim no)
+		(at 288.29 180.594 0)
+		(effects
+			(font
