File: BILLEE_Rover_Control_Module_V1/estop.kicad_sch (KiCad schematic)
At the start: 120 parts, among them CN10 XT60PW-M, CN11 XT60PW-M, CN12 XT90PW-M.G.Y, CN13 XT60PW-M, CN2 XT90PW-M.G.Y, CN3 XT60PW-M, CN4 XT90PW-M.G.Y, CN5 XT60PW-M, CN6 XT60PW-M, CN7 XT60PW-M, CN8 XT60PW-M, CN9 XT60PW-M, Q1 IPT007N06N, Q2 IPT007N06N, Q3 IPT007N06N, Q4 IPT007N06N, Q5 IPT007N06N, Q6 IPT007N06N, Q7 IPT007N06N, Q8 IPT007N06N, U1 Screw Terminal for ESTOP - NO, U11 LTC7001IMSE#PBF, U12 INA780BIDEKR, U13 LTC7001IMSE#PBF, U14 INA780BIDEKR, U26 LTC7001IMSE#PBF, U27 INA780BIDEKR, U28 LTC7001IMSE#PBF, U29 LTC7001IMSE#PBF, U3 SN74LVC08APWR, U30 LTC7001IMSE#PBF, U31 INA780BIDEKR, U32 INA780BIDEKR, U33 INA780BIDEKR, U34 LTC7001IMSE#PBF, U35 LTC7001IMSE#PBF, U36 INA780BIDEKR, U37 INA780BIDEKR, U39 MCP9808T-E/MS, U4 SN74LVC08APWR, U40 MCP9808T-E/MS

Commit message: Biggus Goodies
Parts:
- removed U1: Screw Terminal for ESTOP - NO, PDB_LCSC:CONN-TH_P5.00_KF301-5.0-2P, symbol PDB_LCSC_Libs:KF301-5.0-2P
- added U16: ESTOP, PDB_LCSC:CONN-TH_P5.00_KF301-5.0-2P, symbol PDB_LCSC_Libs:ESTOP
- R24, R48, R49, R50, R51, R52, R53, R54, R55, R56, R57, R58, R60, R70, R71, R73, R74, R75, R76, R77, R78, R79, R80, R81, R82, R83, R84, R85, R86, R87, R88, R89, R90, R91, R92, R93, R94, R95, R96, R97, R98: footprint (none) -> Resistor_SMD:R_0402_1005Metric
Connections:
- net +3.3V_RP2350_VCC: now also U16.1
- net BUFF_E_STOP_STATUS: now also U16.2

Commit message: Fixes
Connections:
- net +3.3V_RP2350_VCC: no longer U36.3 (A1)
- net BUFF_SCL_0: now also U36.3 (A1)
Other:
- moved on the sheet: R91
Changed lines of the file:
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@@
 		)
 	)
-	(text_box "I2C0	INA780x DRIVE5	0x45	A1=VS, A0=VS"
+	(text_box "I2C0	INA780x ARM	0x4C	A1=SCL, A0=GND"
 		(exclude_from_sim no)
-		(at 351.155 76.6967 0)
+		(at 331.47 72.39 0)
 		(size 59.055 3.9483)
 		(margins 0.9525 0.9525 0.9525 0.9525)
@@
 	)
 	(junction
-		(at 393.7 54.61)
-		(diameter 0)
-		(color 0 0 0 0)
-	)
-	(junction
 		(at 276.86 393.7)
 		(diameter 0)
@@
 	)
 	(junction
+		(at 381 35.56)
+		(diameter 0)
+		(color 0 0 0 0)
+	)
+	(junction
 		(at 207.01 118.11)
 		(diameter 0)
@@
 	)
 	(junction
+		(at 393.7 45.72)
+		(diameter 0)
+		(color 0 0 0 0)
+	)
+	(junction
 		(at 227.33 515.62)
 		(diameter 0)
@@
 	)
 	(junction
-		(at 381 35.56)
-		(diameter 0)
-		(color 0 0 0 0)
-	)
-	(junction
 		(at 288.29 129.54)
 		(diameter 0)
@@
 	(wire
 		(pts
-			(xy 290.83 57.15) (xy 292.1 57.15)
+			(xy 274.32 44.45) (xy 274.32 45.72)
 		)
 		(stroke
@@
 	(wire
 		(pts
-			(xy 237.49 208.28) (xy 241.3 208.28)
+			(xy 290.83 57.15) (xy 292.1 57.15)
 		)
 		(stroke
@@
 	(wire
 		(pts
-			(xy 360.68 33.02) (xy 360.68 34.29)
+			(xy 237.49 208.28) (xy 241.3 208.28)
 		)
 		(stroke
@@
 	(wire
 		(pts
-			(xy 237.49 462.28) (xy 241.3 462.28)
+			(xy 360.68 33.02) (xy 360.68 34.29)
 		)
 		(stroke
@@
 	(wire
 		(pts
-			(xy 378.46 110.49) (xy 378.46 121.92)
+			(xy 237.49 462.28) (xy 241.3 462.28)
 		)
 		(stroke
@@
 	(wire
 		(pts
-			(xy 281.94 523.24) (xy 281.94 528.32)
+			(xy 378.46 110.49) (xy 378.46 121.92)
 		)
 		(stroke
@@
 	(wire
 		(pts
-			(xy 219.71 196.85) (xy 219.71 198.12)
+			(xy 281.94 523.24) (xy 281.94 528.32)
 		)
 		(stroke
@@
 	(wire
 		(pts
-			(xy 429.26 68.58) (xy 438.15 68.58)
+			(xy 219.71 196.85) (xy 219.71 198.12)
 		)
 		(stroke
@@
 	(wire
 		(pts
-			(xy 393.7 35.56) (xy 393.7 54.61)
+			(xy 429.26 68.58) (xy 438.15 68.58)
 		)
 		(stroke
@@
 	(wire
 		(pts
-			(xy 274.32 38.1) (xy 274.32 35.56)
+			(xy 274.32 36.83) (xy 274.32 35.56)
 		)
 		(stroke
@@
 	(wire
 		(pts
+			(xy 392.43 35.56) (xy 381 35.56)
+		)
+		(stroke
+			(width 0)
+			(type default)
+		)
+	)
+	(wire
+		(pts
 			(xy 419.1 170.18) (xy 419.1 171.45)
 		)
@@
 	(wire
 		(pts
+			(xy 391.16 54.61) (xy 392.43 54.61)
+		)
+		(stroke
+			(width 0)
+			(type default)
+		)
+	)
+	(wire
+		(pts
 			(xy 290.83 464.82) (xy 293.37 464.82)
 		)
@@
 	(wire
 		(pts
+			(xy 393.7 57.15) (xy 393.7 45.72)
+		)
+		(stroke
+			(width 0)
+			(type default)
+		)
+	)
+	(wire
+		(pts
 			(xy 152.4 461.01) (xy 147.32 461.01)
 		)
@@
 	(wire
 		(pts
-			(xy 393.7 57.15) (xy 391.16 57.15)
+			(xy 391.16 57.15) (xy 393.7 57.15)
 		)
 		(stroke
@@
 	(wire
 		(pts
-			(xy 393.7 54.61) (xy 391.16 54.61)
-		)
-		(stroke
-			(width 0)
-			(type default)
-		)
-	)
-	(wire
-		(pts
 			(xy 237.49 398.78) (xy 241.3 398.78)
 		)
@@
 	(wire
 		(pts
-			(xy 391.16 45.72) (xy 394.97 45.72)
+			(xy 391.16 45.72) (xy 393.7 45.72)
 		)
 		(stroke
@@
 	(wire
 		(pts
-			(xy 393.7 54.61) (xy 393.7 57.15)
-		)
-		(stroke
-			(width 0)
-			(type default)
-		)
-	)
-	(wire
-		(pts
 			(xy 292.1 64.77) (xy 292.1 57.15)
 		)
@@
 	(wire
 		(pts
+			(xy 393.7 45.72) (xy 394.97 45.72)
+		)
+		(stroke
+			(width 0)
+			(type default)
+		)
+	)
+	(wire
+		(pts
 			(xy 80.01 180.34) (xy 80.01 243.84)
 		)
@@
 	(wire
 		(pts
+			(xy 392.43 54.61) (xy 392.43 35.56)
+		)
+		(stroke
+			(width 0)
+			(type default)
+		)
+	)
+	(wire
+		(pts
 			(xy 67.31 74.93) (xy 67.31 80.01)
 		)
@@
 	(wire
 		(pts
-			(xy 381 35.56) (xy 393.7 35.56)
-		)
-		(stroke
-			(width 0)
-			(type default)
-		)
-	)
-	(wire
-		(pts
 			(xy 152.4 397.51) (xy 147.32 397.51)
 		)
@@
 	(symbol
 		(lib_id "Device:R_US")
-		(at 274.32 41.91 180)
+		(at 274.32 40.64 180)
 		(unit 1)
 		(body_style 1)
@@
 		(fields_autoplaced yes)
 		(property "Reference" "R91"
-			(at 276.86 40.6399 0)
+			(at 276.86 39.3699 0)
 			(show_name no)
 			(do_not_autoplace no)
@@
 		)
 		(property "Value" "150k"
-			(at 276.86 43.1799 0)
+			(at 276.86 41.9099 0)
 			(show_name no)
 			(do_not_autoplace no)
@@
 		)
 		(property "Footprint" "Resistor_SMD:R_0402_1005Metric"
-			(at 273.304 41.656 90)
+			(at 273.304 40.386 90)
 			(hide yes)
 			(show_name no)
@@
 		)
 		(property "Datasheet" ""
-			(at 274.32 41.91 0)
+			(at 274.32 40.64 0)
 			(hide yes)
 			(show_name no)
@@
 		)
 		(property "Description" "Resistor, US symbol"
-			(at 274.32 41.91 0)
+			(at 274.32 40.64 0)
 			(hide yes)
 			(show_name no)

Commit message: Schematic Fixed in NO RCP yet
Parts:
- C66, C67, C68, C69, C70, C71: footprint (none) -> Capacitor_SMD:C_0603_1608Metric
Connections:
- net +3.3V_RP2350_VCC: no longer U36.4 (A0)
- net GND: now also U36.4 (A0)
Changed lines of the file:
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@@
 		)
 	)
-	(text_box "I2C0	INA780x DRIVE6	0x47	A1=VS, A0=SCL"
+	(text_box "I2C0	INA780x SCIENCE	0x4D	A1=SCL, A0=VS"
 		(exclude_from_sim no)
 		(at 339.09 136.525 0)
@@
 	)
 	(junction
-		(at 378.46 110.49)
-		(diameter 0)
-		(color 0 0 0 0)
-	)
-	(junction
 		(at 290.83 337.82)
 		(diameter 0)
@@
 	)
 	(junction
-		(at 381 35.56)
-		(diameter 0)
-		(color 0 0 0 0)
-	)
-	(junction
 		(at 207.01 118.11)
 		(diameter 0)
@@
 	)
 	(junction
-		(at 365.76 100.33)
+		(at 398.78 105.41)
 		(diameter 0)
 		(color 0 0 0 0)
 	)
 	(junction
-		(at 398.78 105.41)
+		(at 276.86 203.2)
 		(diameter 0)
 		(color 0 0 0 0)
 	)
 	(junction
-		(at 276.86 203.2)
+		(at 154.94 544.83)
 		(diameter 0)
 		(color 0 0 0 0)
 	)
 	(junction
-		(at 154.94 544.83)
+		(at 365.76 100.33)
 		(diameter 0)
 		(color 0 0 0 0)
@@
 	)
 	(junction
+		(at 378.46 110.49)
+		(diameter 0)
+		(color 0 0 0 0)
+	)
+	(junction
 		(at 162.56 257.81)
 		(diameter 0)
@@
 	(wire
 		(pts
-			(xy 378.46 110.49) (xy 378.46 121.92)
-		)
-		(stroke
-			(width 0)
-			(type default)
-		)
-	)
-	(wire
-		(pts
 			(xy 281.94 523.24) (xy 281.94 528.32)
 		)
@@
 	(wire
 		(pts
-			(xy 392.43 35.56) (xy 381 35.56)
+			(xy 419.1 170.18) (xy 419.1 171.45)
 		)
 		(stroke
@@
 	(wire
 		(pts
-			(xy 419.1 170.18) (xy 419.1 171.45)
+			(xy 391.16 54.61) (xy 392.43 54.61)
 		)
 		(stroke
@@
 	(wire
 		(pts
-			(xy 391.16 54.61) (xy 392.43 54.61)
+			(xy 290.83 464.82) (xy 293.37 464.82)
 		)
 		(stroke
@@
 	(wire
 		(pts
-			(xy 290.83 464.82) (xy 293.37 464.82)
+			(xy 377.19 119.38) (xy 377.19 100.33)
 		)
 		(stroke
@@
 	(wire
 		(pts
-			(xy 365.76 100.33) (xy 377.19 100.33)
-		)
-		(stroke
-			(width 0)
-			(type default)
-		)
-	)
-	(wire
-		(pts
 			(xy 360.68 34.29) (xy 360.68 40.64)
 		)
@@
 	(wire
 		(pts
+			(xy 378.46 110.49) (xy 379.73 110.49)
+		)
+		(stroke
+			(width 0)
+			(type default)
+		)
+	)
+	(wire
+		(pts
 			(xy 180.34 266.7) (xy 207.01 266.7)
 		)
@@
 	(wire
 		(pts
-			(xy 378.46 110.49) (xy 379.73 110.49)
-		)
-		(stroke
-			(width 0)
-			(type default)
-		)
-	)
-	(wire
-		(pts
 			(xy 152.4 270.51) (xy 147.32 270.51)
 		)
@@
 	(wire
 		(pts
-			(xy 377.19 119.38) (xy 377.19 100.33)
-		)
-		(stroke
-			(width 0)
-			(type default)
-		)
-	)
-	(wire
-		(pts
 			(xy 240.03 452.12) (xy 240.03 471.17)
 		)
@@
 	(wire
 		(pts
+			(xy 378.46 110.49) (xy 378.46 121.92)
+		)
+		(stroke
+			(width 0)
+			(type default)
+		)
+	)
+	(wire
+		(pts
 			(xy 358.14 99.06) (xy 358.14 100.33)
 		)
@@
 	(wire
 		(pts
+			(xy 377.19 100.33) (xy 365.76 100.33)
+		)
+		(stroke
+			(width 0)
+			(type default)
+		)
+	)
+	(wire
+		(pts
 			(xy 306.07 31.75) (xy 309.88 31.75)
 		)
@@
 	(wire
 		(pts
-			(xy 392.43 54.61) (xy 392.43 35.56)
-		)
-		(stroke
-			(width 0)
-			(type default)
-		)
-	)
-	(wire
-		(pts
 			(xy 67.31 74.93) (xy 67.31 80.01)
 		)
@@
 	(wire
 		(pts
+			(xy 392.43 54.61) (xy 392.43 58.42)
+		)
+		(stroke
+			(width 0)
+			(type default)
+		)
+	)
+	(wire
+		(pts
 			(xy 209.55 462.28) (xy 209.55 464.82)
 		)
@@
 			)
 		)
-		(property "Footprint" ""
+		(property "Footprint" "Capacitor_SMD:C_0603_1608Metric"
 			(at 414.9852 68.58 0)
 			(hide yes)
@@
 	)
 	(symbol
+		(lib_id "power:GND")
+		(at 392.43 58.42 0)
+		(unit 1)
+		(body_style 1)
+		(exclude_from_sim no)
+		(in_bom yes)
+		(on_board yes)
+		(in_pos_files yes)
+		(dnp no)
+		(property "Reference" "#PWR0200"
+			(at 392.43 64.77 0)
+			(hide yes)
+			(show_name no)
+			(do_not_autoplace no)
+			(effects
+				(font
+					(size 1.27 1.27)
+				)
+			)
+		)
+		(property "Value" "GND"
+			(at 392.43 62.484 0)
+			(show_name no)
+			(do_not_autoplace no)
+			(effects
+				(font
+					(size 1.27 1.27)
+				)
+			)
+		)
+		(property "Footprint" ""
+			(at 392.43 58.42 0)
+			(hide yes)
+			(show_name no)
+			(do_not_autoplace no)
+			(effects
+				(font
+					(size 1.27 1.27)
+				)
+			)
+		)
+		(property "Datasheet" ""
+			(at 392.43 58.42 0)
+			(hide yes)
+			(show_name no)
+			(do_not_autoplace no)
+			(effects
+				(font
+					(size 1.27 1.27)
+				)
+			)
+		)
+		(property "Description" "Power symbol creates a global label with name \"GND\" , ground"
+			(at 392.43 58.42 0)
+			(hide yes)
+			(show_name no)
+			(do_not_autoplace no)
+			(effects
+				(font
+					(size 1.27 1.27)
+				)
+			)
+		)
+		(pin "1"
+		)
+		(instances
+			(project "BILLEE_Rover_Control_Module_V1"
+				(path "/e701dc98-f022-461d-84b5-6b2dd8d89d58/38c7de8f-1e1e-425a-b64c-5257d5cddadc"
+					(reference "#PWR0200")
+					(unit 1)
+				)
+			)
+		)
+	)
+	(symbol
 		(lib_id "power:+3.3V")
 		(at 276.86 201.93 0)
@@
 			)
 		)
-		(property "Footprint" ""
+		(property "Footprint" "Capacitor_SMD:C_0603_1608Metric"
 			(at 417.5252 113.03 0)
 			(hide yes)
@@
 			)
 		)
-		(property "Footprint" ""
+		(property "Footprint" "Capacitor_SMD:C_0603_1608Metric"
 			(at 397.2052 68.58 0)
 			(hide yes)
@@
 			)
 		)
-		(property "Footprint" ""
+		(property "Footprint" "Capacitor_SMD:C_0603_1608Metric"
 			(at 406.0952 68.58 0)
 			(hide yes)
@@
 			)
 		)
-		(property "Footprint" ""
+		(property "Footprint" "Capacitor_SMD:C_0603_1608Metric"
 			(at 399.7452 113.03 0)
 			(hide yes)
@@
 			)
 		)
-		(property "Footprint" ""
+		(property "Footprint" "Capacitor_SMD:C_0603_1608Metric"
 			(at 408.6352 113.03 0)
 			(hide yes)

Commit message: Updated footprint selection
Still missing the four inductors for the regulators, two of them can be poached from scales
Parts:
- C28, C29, C30, C31, C32, C33, C34, C45, C46, C47, C48, C49, C50, C51, C52, C53, C54, C55, C56, C57, C58, C59, C60, C61: footprint Capacitor_SMD:C_0402_1005Metric -> Capacitor_SMD:C_0603_1608Metric
- C66, C67, C68, C69, C70, C71: footprint Capacitor_SMD:C_0603_1608Metric -> Capacitor_SMD:C_1210_3225Metric
Changed lines of the file:
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@@
 			)
 		)
-		(property "Footprint" "Capacitor_SMD:C_0402_1005Metric"
+		(property "Footprint" "Capacitor_SMD:C_0603_1608Metric"
 			(at 92.4052 469.9 0)
 			(hide yes)
@@
 			)
 		)
-		(property "Footprint" "Capacitor_SMD:C_0402_1005Metric"
+		(property "Footprint" "Capacitor_SMD:C_0603_1608Metric"
 			(at 163.5252 459.74 0)
 			(hide yes)
@@
 			)
 		)
-		(property "Footprint" "Capacitor_SMD:C_0402_1005Metric"
+		(property "Footprint" "Capacitor_SMD:C_0603_1608Metric"
 			(at 322.2752 43.18 0)
 			(hide yes)
@@
 			)
 		)
-		(property "Footprint" "Capacitor_SMD:C_0402_1005Metric"
+		(property "Footprint" "Capacitor_SMD:C_0603_1608Metric"
 			(at 92.4052 279.4 0)
 			(hide yes)
@@
 			)
 		)
-		(property "Footprint" "Capacitor_SMD:C_0402_1005Metric"
+		(property "Footprint" "Capacitor_SMD:C_0603_1608Metric"
 			(at 301.9552 107.95 0)
 			(hide yes)
@@
 			)
 		)
-		(property "Footprint" "Capacitor_SMD:C_0402_1005Metric"
+		(property "Footprint" "Capacitor_SMD:C_0603_1608Metric"
 			(at 153.3652 278.13 0)
 			(hide yes)
@@
 			)
 		)
-		(property "Footprint" "Capacitor_SMD:C_0603_1608Metric"
+		(property "Footprint" "Capacitor_SMD:C_1210_3225Metric"
 			(at 414.9852 68.58 0)
 			(hide yes)
@@
 			)
 		)
-		(property "Footprint" "Capacitor_SMD:C_0402_1005Metric"
+		(property "Footprint" "Capacitor_SMD:C_0603_1608Metric"
 			(at 153.3652 341.63 0)
 			(hide yes)
@@
 			)
 		)
-		(property "Footprint" "Capacitor_SMD:C_0603_1608Metric"
+		(property "Footprint" "Capacitor_SMD:C_1210_3225Metric"
 			(at 417.5252 113.03 0)
 			(hide yes)
@@
 			)
 		)
-		(property "Footprint" "Capacitor_SMD:C_0402_1005Metric"
+		(property "Footprint" "Capacitor_SMD:C_0603_1608Metric"
 			(at 230.8352 118.11 0)
 			(hide yes)
@@
 			)
 		)
-		(property "Footprint" "Capacitor_SMD:C_0603_1608Metric"
+		(property "Footprint" "Capacitor_SMD:C_1210_3225Metric"
 			(at 397.2052 68.58 0)
 			(hide yes)
@@
 			)
 		)
-		(property "Footprint" "Capacitor_SMD:C_0402_1005Metric"
+		(property "Footprint" "Capacitor_SMD:C_0603_1608Metric"
 			(at 163.5252 332.74 0)
 			(hide yes)
@@
 			)
 		)
-		(property "Footprint" "Capacitor_SMD:C_0603_1608Metric"
+		(property "Footprint" "Capacitor_SMD:C_1210_3225Metric"
 			(at 406.0952 68.58 0)
 			(hide yes)
@@
 			)
 		)
-		(property "Footprint" "Capacitor_SMD:C_0402_1005Metric"
+		(property "Footprint" "Capacitor_SMD:C_0603_1608Metric"
 			(at 92.4052 533.4 0)
 			(hide yes)
@@
 			)
 		)
-		(property "Footprint" "Capacitor_SMD:C_0402_1005Metric"
+		(property "Footprint" "Capacitor_SMD:C_0603_1608Metric"
 			(at 153.3652 532.13 0)
 			(hide yes)
@@
 			)
 		)
-		(property "Footprint" "Capacitor_SMD:C_0603_1608Metric"
+		(property "Footprint" "Capacitor_SMD:C_1210_3225Metric"
 			(at 399.7452 113.03 0)
 			(hide yes)
@@
 			)
 		)
-		(property "Footprint" "Capacitor_SMD:C_0402_1005Metric"
+		(property "Footprint" "Capacitor_SMD:C_0603_1608Metric"
 			(at 251.1552 53.34 0)
 			(hide yes)
@@
 			)
 		)
-		(property "Footprint" "Capacitor_SMD:C_0402_1005Metric"
+		(property "Footprint" "Capacitor_SMD:C_0603_1608Metric"
 			(at 153.3652 468.63 0)
 			(hide yes)
@@
 			)
 		)
-		(property "Footprint" "Capacitor_SMD:C_0402_1005Metric"
+		(property "Footprint" "Capacitor_SMD:C_0603_1608Metric"
 			(at 312.1152 52.07 0)
 			(hide yes)
@@
 			)
 		)
-		(property "Footprint" "Capacitor_SMD:C_0402_1005Metric"
+		(property "Footprint" "Capacitor_SMD:C_0603_1608Metric"
 			(at 92.4052 406.4 0)
 			(hide yes)
@@
 			)
 		)
-		(property "Footprint" "Capacitor_SMD:C_0402_1005Metric"
+		(property "Footprint" "Capacitor_SMD:C_0603_1608Metric"
 			(at 92.4052 342.9 0)
 			(hide yes)
@@
 			)
 		)
-		(property "Footprint" "Capacitor_SMD:C_0402_1005Metric"
+		(property "Footprint" "Capacitor_SMD:C_0603_1608Metric"
 			(at 163.5252 523.24 0)
 			(hide yes)
@@
 			)
 		)
-		(property "Footprint" "Capacitor_SMD:C_0402_1005Metric"
+		(property "Footprint" "Capacitor_SMD:C_0603_1608Metric"
 			(at 163.5252 205.74 0)
 			(hide yes)
@@
 			)
 		)
-		(property "Footprint" "Capacitor_SMD:C_0402_1005Metric"
+		(property "Footprint" "Capacitor_SMD:C_0603_1608Metric"
 			(at 92.4052 215.9 0)
 			(hide yes)
@@
 			)
 		)
-		(property "Footprint" "Capacitor_SMD:C_0402_1005Metric"
+		(property "Footprint" "Capacitor_SMD:C_0603_1608Metric"
 			(at 153.3652 214.63 0)
 			(hide yes)
@@
 			)
 		)
-		(property "Footprint" "Capacitor_SMD:C_0402_1005Metric"
+		(property "Footprint" "Capacitor_SMD:C_0603_1608Metric"
 			(at 153.3652 405.13 0)
 			(hide yes)
@@
 			)
 		)
-		(property "Footprint" "Capacitor_SMD:C_0402_1005Metric"
+		(property "Footprint" "Capacitor_SMD:C_0603_1608Metric"
 			(at 291.7952 116.84 0)
 			(hide yes)
@@
 			)
 		)
-		(property "Footprint" "Capacitor_SMD:C_0603_1608Metric"
+		(property "Footprint" "Capacitor_SMD:C_1210_3225Metric"
 			(at 408.6352 113.03 0)
 			(hide yes)
@@
 			)
 		)
-		(property "Footprint" "Capacitor_SMD:C_0402_1005Metric"
+		(property "Footprint" "Capacitor_SMD:C_0603_1608Metric"
 			(at 163.5252 396.24 0)
 			(hide yes)
@@
 			)
 		)
-		(property "Footprint" "Capacitor_SMD:C_0402_1005Metric"
+		(property "Footprint" "Capacitor_SMD:C_0603_1608Metric"
 			(at 163.5252 269.24 0)
 			(hide yes)

Commit message: Updated reference designators. Schematic Complete
Not including RCP for Drivetrain/Arm/Science
Parts:
- renumbered C30 to C42, C49 to C43, C48 to C44, C47 to C45, C34 to C46, C31 to C47, C28 to C48, C32 to C49, C45 to C50, C50 to C51, C51 to C52, C52 to C53, C29 to C54, C33 to C55, C46 to C56, C53 to C57, C54 to C58, C55 to C59, C57 to C60, C56 to C61, C59 to C62, C61 to C63, C58 to C64, C60 to C65, C69 to C67, C67 to C68, C70 to C69, C68 to C70, CN3 to CN10, CN5 to CN11, CN6 to CN12, CN7 to CN13, CN8 to CN14, CN9 to CN15, CN11 to CN16, CN10 to CN17, CN13 to CN18, CN2 to CN7, CN12 to CN8, CN4 to CN9, D9 to D10, D8 to D11, D2 to D4, D3 to D5, D4 to D6, D5 to D7, D6 to D8, D7 to D9, Q8 to Q7, Q7 to Q8, R86 to R100, R88 to R101, R90 to R61, R49 to R62, R50 to R63, R51 to R64, R52 to R65, R55 to R66, R56 to R67, R60 to R68, R70 to R69, R71 to R70, R73 to R71, R74 to R72, R75 to R73, R93 to R74, R94 to R75, R95 to R76, R98 to R77, R96 to R78, R97 to R79, R24 to R80, R53 to R81, R57 to R82, R76 to R83, R77 to R84, R78 to R85, R48 to R86, R54 to R87, R58 to R88, R79 to R89, R80 to R90, R81 to R91, R84 to R92, R85 to R93, R92 to R94, R82 to R95, R83 to R96, R91 to R97, R87 to R98, R89 to R99, U3 to U17, U4 to U18, U11 to U19, U13 to U20, U26 to U21, U28 to U22, U29 to U23, U30 to U24, U12 to U25, U14 to U26, U31 to U28, U32 to U29, U33 to U30, U35 to U31, U34 to U32, U37 to U33, U36 to U34, U39 to U35, U40 to U36

Commit message: Layout...
Parts:
- added C73, C74, C75, C76, C77, C78, C79, C80: 0.1u, Capacitor_SMD:C_0603_1608Metric, symbol Device:C
Connections:
- net +3.3V_RP2350_VCC: now also C73.2, C74.2, C75.2, C76.2, C77.2, C78.2, C79.2, C80.2
- net GND: now also C73.1, C74.1, C75.1, C76.1, C77.1, C78.1, C79.1, C80.1

Commit message: Layout! 🍋
Other:
- moved on the sheet: C75
