File: BILLEE_Rover_Control_Module_V1/estop.kicad_sch (KiCad schematic)
At the start: 128 parts, among them CN10 XT60PW-M, CN11 XT60PW-M, CN12 XT60PW-M, CN13 XT60PW-M, CN14 XT60PW-M, CN15 XT60PW-M, CN16 XT60PW-M, CN17 XT60PW-M, CN18 XT60PW-M, CN7 XT90PW-M.G.Y, CN8 XT90PW-M.G.Y, CN9 XT90PW-M.G.Y, Q1 IPT007N06N, Q2 IPT007N06N, Q3 IPT007N06N, Q4 IPT007N06N, Q5 IPT007N06N, Q6 IPT007N06N, Q7 IPT007N06N, Q8 IPT007N06N, U16 ESTOP, U17 SN74LVC08APWR, U18 SN74LVC08APWR, U19 LTC7001IMSE#PBF, U20 LTC7001IMSE#PBF, U21 LTC7001IMSE#PBF, U22 LTC7001IMSE#PBF, U23 LTC7001IMSE#PBF, U24 LTC7001IMSE#PBF, U25 INA780BIDEKR, U26 INA780BIDEKR, U27 INA780BIDEKR, U28 INA780BIDEKR, U29 INA780BIDEKR, U30 INA780BIDEKR, U31 LTC7001IMSE#PBF, U32 LTC7001IMSE#PBF, U33 INA780BIDEKR, U34 INA780BIDEKR, U35 MCP9808T-E/MS, U36 MCP9808T-E/MS

Commit message: Layout!
Parts:
- C48, C49, C50, C51, C52, C53, C62, C64: Voltage (none) -> 25V
Other:
- moved on the sheet: C60, C62, C63, C67, C69, C71, C79, CN16, CN8, D10, Q7, R92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

Commit message: More layout :tired_face:
Changed lines of the file:
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@@
 	(text_box "I2C0	INA780x SCIENCE	0x4D	A1=SCL, A0=VS"
 		(exclude_from_sim no)
-		(at 365.887 127.3697 0)
+		(at 324.485 138.5457 0)
 		(size 59.055 3.9483)
 		(margins 0.9525 0.9525 0.9525 0.9525)
@@
 	(text_box "AND Gate array for ESTOP Circuit"
 		(exclude_from_sim no)
-		(at 121.92 42.7624 0)
+		(at 69.342 33.1104 0)
 		(size 17.78 8.0376)
 		(margins 0.9525 0.9525 0.9525 0.9525)
@@
 		(exclude_from_sim no)
 		(at 237.49 22.86 0)
-		(size 15.24 15.24)
-		(margins 0.9525 0.9525 0.9525 0.9525)
-		(stroke
+		(size 15.24 12.1268)
+		(margins 0.9525 0.9525 0.9525 0.9525)
+		(stroke

Commit message: Done I think
Parts:
- C42, C43, C44, C45, C46, C47, C60, C61, C66, C67, C68, C69, C70, C71: value 47u -> 10u
- R62, R64, R66, R68, R70, R72, R92, R95: value 840k -> 866k
- R63, R65, R67, R69, R71, R73, R93, R96: value 33k -> 34k
Changed lines of the file:
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@@
 		)
 	)
-	(text_box "Configuring OVLO to be 32v.\nR82 = 840k\nR83 = 33k\n"
+	(text_box "Configuring OVLO to be 32v.\nR82 = 866k\nR83 = 34k\n"
 		(exclude_from_sim no)
 		(at 264.795 56.5928 0)
@@
 			)
 		)
-		(property "Value" "47u"
+		(property "Value" "10u"
 			(at 94.361 467.233 0)
 			(show_name no)
@@
 			)
 		)
-		(property "Value" "47u"
+		(property "Value" "10u"
 			(at 94.361 276.733 0)
 			(show_name no)
@@
 			)
 		)
-		(property "Value" "47u"
+		(property "Value" "10u"
 			(at 420.37 64.516 0)
 			(show_name no)
@@
 			)
 		)
-		(property "Value" "47u"
+		(property "Value" "10u"
 			(at 414.02 112.776 0)
 			(show_name no)
@@
 			)
 		)
-		(property "Value" "47u"
+		(property "Value" "10u"
 			(at 223.901 119.253 0)
 			(show_name no)
@@
 			)
 		)
-		(property "Value" "47u"
+		(property "Value" "10u"
 			(at 402.59 64.516 0)
 			(show_name no)
@@
 			)
 		)
-		(property "Value" "33k"
+		(property "Value" "34k"
 			(at 104.14 344.1699 0)
 			(show_name no)
@@
 			)
 		)
-		(property "Value" "33k"
+		(property "Value" "34k"
 			(at 104.14 471.1699 0)
 			(show_name no)
@@
 			)
 		)
-		(property "Value" "33k"
+		(property "Value" "34k"
 			(at 104.14 534.6699 0)
 			(show_name no)
@@
 			)
 		)
-		(property "Value" "840k"
+		(property "Value" "866k"
 			(at 104.14 336.5499 0)
 			(show_name no)
@@
 			)
 		)
-		(property "Value" "47u"
+		(property "Value" "10u"
 			(at 411.48 64.516 0)
 			(show_name no)
@@
 			)
 		)
-		(property "Value" "47u"
+		(property "Value" "10u"
 			(at 94.361 530.733 0)
 			(show_name no)
@@
 			)
 		)
-		(property "Value" "47u"
+		(property "Value" "10u"
 			(at 396.24 112.776 0)
 			(show_name no)
@@
 			)
 		)
-		(property "Value" "47u"
+		(property "Value" "10u"
 			(at 253.111 50.673 0)
 			(show_name no)
@@
 			)
 		)
-		(property "Value" "840k"
+		(property "Value" "866k"
 			(at 233.68 115.5699 0)
 			(show_name no)
@@
 			)
 		)
-		(property "Value" "47u"
+		(property "Value" "10u"
 			(at 94.361 403.733 0)
 			(show_name no)
@@
 			)
 		)
-		(property "Value" "840k"
+		(property "Value" "866k"
 			(at 104.14 400.0499 0)
 			(show_name no)
@@
 			)
 		)
-		(property "Value" "47u"
+		(property "Value" "10u"
 			(at 94.361 340.233 0)
 			(show_name no)
@@
 			)
 		)
-		(property "Value" "33k"
+		(property "Value" "34k"
 			(at 233.68 123.1899 0)
 			(show_name no)
@@
 			)
 		)
-		(property "Value" "33k"
+		(property "Value" "34k"
 			(at 104.14 280.6699 0)
 			(show_name no)
@@
 			)
 		)
-		(property "Value" "840k"
+		(property "Value" "866k"
 			(at 104.14 273.0499 0)
 			(show_name no)
@@
 			)
 		)
-		(property "Value" "840k"
+		(property "Value" "866k"
 			(at 104.14 209.5499 0)
 			(show_name no)
@@
 			)
 		)
-		(property "Value" "840k"
+		(property "Value" "866k"
 			(at 262.89 46.9899 0)
 			(show_name no)
@@
 			)
 		)
-		(property "Value" "47u"
+		(property "Value" "10u"
 			(at 94.361 213.233 0)
 			(show_name no)
@@
 			)
 		)
-		(property "Value" "840k"
+		(property "Value" "866k"
 			(at 104.14 463.5499 0)
 			(show_name no)
@@
 			)
 		)
-		(property "Value" "840k"
+		(property "Value" "866k"
 			(at 104.14 527.0499 0)
 			(show_name no)
@@
 			)
 		)
-		(property "Value" "47u"
+		(property "Value" "10u"
 			(at 405.13 112.776 0)
 			(show_name no)
@@
 			)
 		)
-		(property "Value" "33k"
+		(property "Value" "34k"
 			(at 104.14 407.6699 0)
 			(show_name no)
@@
 			)
 		)
-		(property "Value" "33k"
+		(property "Value" "34k"
 			(at 262.89 54.6099 0)
 			(show_name no)
@@
 			)
 		)
-		(property "Value" "33k"
+		(property "Value" "34k"
 			(at 104.14 217.1699 0)
 			(show_name no)

Commit message: Updated with Claude Notes. Checking again.
Changed lines of the file:
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@@
 		)
 	)
-	(text_box "Pull down resistor. ESTOP is Normnally Open, so ESTOP OPEN = Pull down Resistor to GND on ALL And Gate `B` inputs."
+	(text_box "ESTOP is Normnally CLOSED, so when ESTOP is pressed = Pull down Resistor to GND on ALL And Gate `B` inputs."
 		(exclude_from_sim no)
 		(at 22.225 34.925 0)

Commit message: Updated Arm/Science rails to be 22.2V not 14.4V. this was a wrong architectural decision that needed updating.
Connections:
- net +14.4V_ARM renamed +22.2V_ARM
- net +14.4V_ARM_BATT renamed +22.2V_ARM_BATT
- net +14.4V_ARM_SENSOR_OUT renamed +22.2V_ARM_SENSOR_OUT
- net +14.4V_SCIENCE renamed +22.2V_SCIENCE
- net +14.4V_SCIENCE_BATT renamed +22.2V_SCIENCE_BATT
- net +14.4V_SCIENCE_SENSOR_OUT renamed +22.2V_SCIENCE_SENSOR_OUT
Changed lines of the file:
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@@
 			)
 		)
-		(property "Value" "+14.4V_SCIENCE"
-			(at 336.55 96.52 0)
+		(property "Value" "+22.2V_SCIENCE"
+			(at 339.09 100.3299 0)
 			(show_name no)
 			(do_not_autoplace no)
@@
 					(size 1.27 1.27)
 				)
+				(justify left)
 			)
 		)
@@
 		(in_pos_files yes)
 		(dnp no)
-		(fields_autoplaced yes)
 		(property "Reference" "#PWR0140"
 			(at 210.82 48.26 0)
@@
 			)
 		)
-		(property "Value" "+14.4V_ARM_BATT"
-			(at 210.82 39.37 0)
+		(property "Value" "+22.2V_ARM_BATT"
+			(at 202.946 39.37 0)
 			(show_name no)
 			(do_not_autoplace no)
@@
 					(size 1.27 1.27)
 				)
+				(justify left)
 			)
 		)
@@
 			)
 		)
-		(property "Value" "+14.4V_ARM_SENSOR_OUT"
+		(property "Value" "+22.2V_ARM_SENSOR_OUT"
 			(at 421.132 34.798 0)
 			(show_name no)
@@
 			)
 		)
-		(property "Value" "+14.4V_ARM"
-			(at 360.68 27.94 0)
+		(property "Value" "+22.2V_ARM"
+			(at 363.22 31.7499 0)
 			(show_name no)
 			(do_not_autoplace no)
@@
 					(size 1.27 1.27)
 				)
+				(justify left)
 			)
 		)
@@
 			)
 		)
-		(property "Value" "+14.4V_SCIENCE_SENSOR_OUT"
+		(property "Value" "+22.2V_SCIENCE_SENSOR_OUT"
 			(at 413.512 103.378 0)
 			(show_name no)
@@
 			)
 		)
-		(property "Value" "+14.4V_SCIENCE_BATT"
+		(property "Value" "+22.2V_SCIENCE_BATT"
 			(at 181.102 109.22 0)
 			(show_name no)
