File: BILLEE_Rover_Control_Module_V1/BILLEE_Rover_Control_Module_V1.kicad_pcb (KiCad board)
At the start: 2 copper layers, 259 parts, among them CN1 XT90PW-M.G.Y, CN10 XT60PW-M, CN11 XT60PW-M, CN12 XT60PW-M, CN13 XT60PW-M, CN14 XT60PW-M, CN15 XT60PW-M, CN16 XT60PW-M, CN17 XT60PW-M, CN18 XT60PW-M, CN2 XT60PW-M, CN3 XT60PW-M, CN4 XT60PW-M, CN5 XT60PW-M, CN6 DF11-18DP-2DSA, CN7 XT90PW-M.G.Y, CN8 XT90PW-M.G.Y, CN9 XT90PW-M.G.Y, J1 2.54mm Header, Q1 IPT007N06N, Q2 IPT007N06N, Q3 IPT007N06N, Q4 IPT007N06N, Q5 IPT007N06N, Q6 IPT007N06N, Q7 IPT007N06N, Q8 IPT007N06N, SW1 33uH, SW2 KMR2, SW3 RESET SW, U1 INA780BIDEKR, U10 RP2350A_C42411118, U11 ABM8-272-T3_C20625731, U12 W25Q128JVSIQTR, U13 TCA4307DGKR, U14 TCA4307DGKR, U15 TXS0108EPWR, U16 ESTOP, U17 SN74LVC08APWR, U18 SN74LVC08APWR, U19 LTC7001IMSE#PBF, U2 MCP9808T-E/MS, U20 LTC7001IMSE#PBF, U21 LTC7001IMSE#PBF, U22 LTC7001IMSE#PBF, U23 LTC7001IMSE#PBF, U24 LTC7001IMSE#PBF, U25 INA780BIDEKR, U26 INA780BIDEKR, U27 INA780BIDEKR, U28 INA780BIDEKR, U29 INA780BIDEKR, U3 TPS1HA08BQPWPRQ1, U30 INA780BIDEKR, U31 LTC7001IMSE#PBF, U32 LTC7001IMSE#PBF, U33 INA780BIDEKR, U34 INA780BIDEKR, U35 MCP9808T-E/MS, U36 MCP9808T-E/MS, U4 TPS1HA08BQPWPRQ1, U5 TPS1HA08BQPWPRQ1, U6 LT8612EUDE#TRPBF, U7 LT8612EUDE#TRPBF, U8 LT8612EUDE#TRPBF, U9 10uH

Commit message: Layout...
Parts:
- added C72: 0.1u, Capacitor_SMD:C_0603_1608Metric, F.Cu at (174.0, 54.5)
- added C73: 0.1u, Capacitor_SMD:C_0603_1608Metric, F.Cu at (18.1, -11.1)
- added C74: 0.1u, Capacitor_SMD:C_0603_1608Metric, F.Cu at (18.1, -8.59)
- added C75: 0.1u, Capacitor_SMD:C_0603_1608Metric, F.Cu at (18.1, -6.08)
- added C76: 0.1u, Capacitor_SMD:C_0603_1608Metric, F.Cu at (18.1, -3.56)
- added C77: 0.1u, Capacitor_SMD:C_0603_1608Metric, F.Cu at (18.1, -1.05)
- added C78: 0.1u, Capacitor_SMD:C_0603_1608Metric, F.Cu at (18.1, 1.46)
- added C79: 0.1u, Capacitor_SMD:C_0603_1608Metric, F.Cu at (18.1, 3.96)
- added C80: 0.1u, Capacitor_SMD:C_0603_1608Metric, F.Cu at (18.1, 6.47)
- C20, C23: footprint Capacitor_SMD:C_1210_3225Metric -> Capacitor_SMD:C_01005_0402Metric
- TP1, TP2, TP3, TP4, TP5, TP6: footprint Connector_Pin:Pin_D1.0mm_L10.0mm -> TestPoint:TestPoint_THTPad_2.0x2.0mm_Drill1.0mm
- moved Q7 358.6 mm to (416.4, 81.1)
- moved CN16 332.8 mm to (425.9, 63.9)
- moved CN8 327.4 mm to (400.8, 76.0)
- moved C71 314.1 mm to (427.0, 82.8)
- moved C69 313.9 mm to (427.0, 78.6)
- moved D10 313.7 mm to (417.7, 90.9)
- moved C67 313.7 mm to (427.0, 74.3)
- moved C62 279.0 mm to (402.8, 88.0)
- moved C63 279.0 mm to (402.8, 90.5)
- moved U31 279.0 mm to (406.9, 87.6)
- moved C60 278.8 mm to (402.8, 85.5)
- moved CN17 277.4 mm to (368.4, 65.4)
- moved CN18 277.4 mm to (368.4, 82.2)
- moved Q8 267.2 mm to (336.4, 94.7)
- moved U33 266.7 mm to (397.1, 88.2)
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Routing:
- net +3.3V_RP2350_VCC: track 0.00 -> 24.4 mm, vias 0 -> 4
- net +22.2V_LOGIC_POWER_SENSOR_OUT: track 0.00 -> 18.5 mm, vias 0 -> 2
- net GND: track 0.00 -> 9.29 mm, vias 0 -> 33
- net Net-(U4-VOUT): track 0.00 -> 6.62 mm
- net Net-(U7-EN/UV): track 0.00 -> 5.97 mm, vias 0 -> 2
- net Net-(D2-A): track 0.00 -> 4.70 mm, vias 0 -> 2
- net Net-(U4-EN): track 0.00 -> 4.70 mm, vias 0 -> 2
- net Net-(U7-RT): track 0.00 -> 4.01 mm
- net Net-(U4-DIA_EN): track 0.00 -> 3.59 mm, vias 0 -> 2
- net Net-(U7-BST): track 0.00 -> 3.19 mm
- net +22.2V_LOGIC: track 0.00 -> 2.85 mm
- net Net-(U7-TR/SS): track 0.00 -> 2.23 mm, vias 0 -> 2
- net Net-(U4-LATCH): track 0.00 -> 1.82 mm
- net Net-(U4-SNS): track 0.00 -> 1.62 mm
- net Net-(U4-SEL1): track 0.00 -> 1.56 mm
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- added copper zone on F.Cu, net +22.2V_LOGIC_POWER_SENSOR_OUT
- added copper zone on F.Cu, net Net-(U4-VOUT)
- added copper zone on F.Cu, net Net-(U7-FB)
- added copper zone on F.Cu, net Net-(U7-SW)
Other:
- copper layers 2 -> 4
- board text added: "C2150178"

Commit message: continuing layout
Parts:
- U15: moved to B.Cu
- moved CN10 316.5 mm to (248.0, 115.0), turned to 180 degrees
- moved CN11 299.6 mm to (248.0, 98.3), turned to 180 degrees
- moved Q1 299.5 mm to (238.1, 114.5), turned to 180 degrees
- moved U25 287.4 mm to (237.8, 104.0), turned to 180 degrees
- moved CN12 285.6 mm to (248.0, 81.5), turned to 180 degrees
- moved Q2 279.9 mm to (226.0, 114.5), turned to 180 degrees
- moved U26 279.5 mm to (237.8, 96.1), turned to 180 degrees
- moved CN13 275.1 mm to (248.0, 64.8), turned to 180 degrees
- moved D4 272.5 mm to (228.5, 104.7), turned to 180 degrees
- moved U27 272.3 mm to (237.8, 88.2), turned to 180 degrees
- moved CN14 268.3 mm to (248.0, 48.0), turned to 180 degrees
- moved D5 266.2 mm to (228.5, 99.0), turned to 180 degrees
- moved U28 265.8 mm to (237.8, 80.3), turned to 180 degrees
- moved CN15 265.6 mm to (248.0, 31.3), turned to 180 degrees
- moved Q3 261.1 mm to (213.8, 114.5), turned to 180 degrees
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Routing:
- net +1V1: track 0.00 -> 20.3 mm
- net /RP2350A/QSPI_SS: track 0.00 -> 10.6 mm
- net /RP2350A/QSPI_SD2: track 0.00 -> 9.79 mm, vias 0 -> 2
- net /RP2350A/QSPI_SD1: track 0.00 -> 9.77 mm
- net GND: track 9.29 -> 18.5 mm, vias 33 -> 85
- net +22.2V_POE_VCC: track 0.00 -> 7.82 mm
- net /RP2350A/XOUT_R: track 0.00 -> 6.78 mm
- net Net-(U6-EN/UV): track 0.00 -> 6.42 mm, vias 0 -> 2
- net /RP2350A/RUN: track 0.00 -> 6.23 mm
- net /RP2350A/~{USB_BOOT}: track 0.00 -> 5.82 mm
- net +22.2V_LOGIC_POWER_SENSOR_OUT: track 18.5 -> 24.3 mm, vias 2 -> 4
- net /RP2350A/QSPI_SD3: track 0.00 -> 5.72 mm
- net /RP2350A/SW_RUN_R: track 0.00 -> 5.51 mm
- net +20V_JETSON_VCC: track 0.00 -> 4.37 mm, vias 0 -> 2
- net /RP2350A/FLASH_SS: track 0.00 -> 4.30 mm
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- added copper zone on F.Cu, net +20V_JETSON_VCC
- added copper zone on F.Cu, net +22.2V_LOGIC
- added copper zone on F.Cu, net +22.2V_POE_VCC
- added copper zone on F.Cu, net Net-(U6-FB)
- added copper zone on F.Cu, net Net-(U6-SW)

Commit message: Layout Cont.
Parts:
- removed TP2: TestPoint, TestPoint:TestPoint_THTPad_2.0x2.0mm_Drill1.0mm
- added H1: MountingHole_Pad, MountingHole:MountingHole_5.3mm_M5_Pad_Via, F.Cu at (66.8, 25.6)
- added H2: MountingHole_Pad, MountingHole:MountingHole_5.3mm_M5_Pad_Via, F.Cu at (66.8, 37.7)
- added H3: MountingHole_Pad, MountingHole:MountingHole_5.3mm_M5_Pad_Via, F.Cu at (66.8, 49.9)
- added H4: MountingHole_Pad, MountingHole:MountingHole_5.3mm_M5_Pad_Via, F.Cu at (66.8, 62.0)
- C2, C72, R57, R58: moved to B.Cu
- moved R48 211.2 mm to (243.6, -23.3)
- moved R50 209.7 mm to (243.5, -15.8)
- moved R56 207.5 mm to (241.6, -23.3), turned to 180 degrees
- moved R60 203.8 mm to (244.7, -19.4), turned to -90 degrees
- moved R47 203.3 mm to (235.9, -23.2)
- moved R54 202.9 mm to (241.5, -15.8), turned to 180 degrees
- moved R49 201.9 mm to (235.9, -15.8)
- moved R52 201.9 mm to (240.5, -19.4), turned to 90 degrees
- moved R55 199.6 mm to (233.9, -23.2), turned to 180 degrees
- moved R59 195.9 mm to (237.0, -19.4), turned to -90 degrees
- moved R53 195.1 mm to (233.9, -15.8), turned to 180 degrees
- moved U14 194.9 mm to (242.6, -19.5)
- moved R51 193.9 mm to (232.8, -19.3), turned to 90 degrees
- moved U13 192.2 mm to (234.9, -19.5)
- moved U35 183.4 mm to (204.8, -18.7)
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Connections:
- CN4 pad 3: Net-(CN4-Pad3) -> GND
- CN4 pad 4: Net-(CN4-Pad3) -> GND
Routing:
- net +3.3V_RP2350_VCC: track 24.4 -> 127.2 mm, vias 4 -> 9
- net BUFF_E_STOP_STATUS: track 3.19 -> 40.8 mm, vias 0 -> 3
- net /RP2350A/~{USB_BOOT}: track 5.82 -> 21.5 mm, vias 0 -> 2
- net /RP2350A/SWCLK: track 0.00 -> 13.5 mm, vias 0 -> 1
- net /RP2350A/SWD: track 0.00 -> 10.2 mm, vias 0 -> 1
- net GND: track 18.5 -> 27.9 mm, vias 85 -> 141
- net Net-(U5-VOUT): track 0.00 -> 8.44 mm
- net USB_D+: track 0.00 -> 7.99 mm
- net USB_D-: track 0.00 -> 7.97 mm
- net /RP2350A/DP_D-: track 0.00 -> 7.94 mm
- net /RP2350A/DP_D+: track 0.00 -> 7.93 mm
- net Net-(D2-A): track 2.86 -> 10.3 mm, vias 1 -> 2
- net VBUS_USB: track 0.00 -> 7.30 mm
- net BUFF_DRIVE_EN_4: track 0.00 -> 5.39 mm, vias 0 -> 1
- net +22.2V_LOGIC_POWER_SENSOR_OUT: track 24.3 -> 19.0 mm, vias 4 -> 5
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- added copper zone on F.Cu, net +12V_AUX_VCC
- added copper zone on F.Cu, net +3.3V_RP2350_VCC
- added copper zone on F.Cu, net Net-(U5-VOUT)
- added copper zone on F.Cu, net Net-(U8-FB)
- added copper zone on F.Cu, net Net-(U8-SW)

Commit message: Layout! 🍋
Parts:
- H1, H2, H3, H4: footprint MountingHole:MountingHole_5.3mm_M5_Pad_Via -> MountingHole:MountingHole_4.3mm_M4_Pad_Via
- R22, R24, R26: value 180k -> 200k
- moved CN7 191.9 mm to (122.9, 72.5), turned to 0 degrees
- moved U35 143.8 mm to (145.2, 112.1), turned to 90 degrees
- moved U36 141.7 mm to (145.2, 107.7), turned to 90 degrees
- moved R55 141.3 mm to (140.8, 83.0), turned to -90 degrees
- moved R48 141.2 mm to (140.7, 73.3), turned to 90 degrees
- moved R56 141.1 mm to (140.7, 75.3), turned to -90 degrees
- moved R47 141.1 mm to (140.8, 81.0), turned to 90 degrees
- moved U13 135.9 mm to (144.5, 82.0), turned to 90 degrees
- moved R51 135.9 mm to (144.6, 84.1), turned to 180 degrees
- moved U14 135.8 mm to (144.5, 74.3), turned to 90 degrees
- moved R60 135.7 mm to (144.5, 72.2), turned to 0 degrees
- moved R59 135.7 mm to (144.6, 79.9), turned to 0 degrees
- moved R52 135.6 mm to (144.6, 76.4), turned to 180 degrees
- moved CN16 135.1 mm to (173.0, 47.1), turned to 90 degrees
- moved R95 132.3 mm to (167.4, 94.3), turned to 90 degrees
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Routing:
- net GND: track 27.9 -> 50.2 mm, vias 141 -> 138
- net /RP2350A/SWCLK: track 13.5 -> 0.62 mm
- net +12V_AUX_VCC: track 0.00 -> 12.9 mm
- net /RP2350A/QSPI_SD2: track 9.79 -> 1.28 mm
- net /RP2350A/SWD: track 10.2 -> 1.74 mm
- net Net-(U6-EN/UV): track 6.42 -> 1.06 mm
- net +22.2V_LOGIC: track 2.85 -> 0.00 mm
- net Net-(U1-IN–): track 0.95 -> 0.00 mm
- net Net-(U1-IN+): track 0.75 -> 0.00 mm
- net +3.3V_RP2350_VCC: vias 9 -> 7
- net +22.2V_LOGIC_POWER_SENSOR_OUT: vias 5 -> 4
- removed copper zone on F.Cu, net +22.2V_LOGIC

Commit message: Layout!
Parts:
- moved H2 246.0 mm to (257.4, 45.0)
- moved H3 240.4 mm to (258.3, 117.3)
- moved CN10 117.5 mm to (190.1, 52.6), turned to -90 degrees
- moved U25 105.0 mm to (193.2, 62.3), turned to 180 degrees
- moved C42 100.1 mm to (185.3, 59.1), turned to 0 degrees
- moved C76 98.7 mm to (197.7, 61.5), turned to -90 degrees
- moved R74 96.2 mm to (187.8, 59.5), turned to 180 degrees
- moved R62 96.0 mm to (184.8, 60.4), turned to 180 degrees
- moved R63 96.0 mm to (184.8, 61.5), turned to 0 degrees
- moved CN8 95.5 mm to (90.5, 59.3), turned to 0 degrees
- moved R86 93.7 mm to (184.8, 62.6), turned to 0 degrees
- moved U19 93.2 mm to (187.3, 63.1), turned to 180 degrees
- moved D4 93.2 mm to (181.7, 63.4)
- moved D10 91.8 mm to (114.2, 87.9), turned to -90 degrees
- moved CN11 91.8 mm to (210.7, 52.6), turned to -90 degrees
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Routing:
- net +3.3V_RP2350_VCC: track 127.2 -> 164.4 mm
- net GND: track 50.2 -> 27.9 mm, vias 138 -> 192
- net /RP2350A/~{USB_BOOT}: track 21.5 -> 4.10 mm
- net +12V_AUX_VCC: track 12.9 -> 0.00 mm
- net BUFF_SCL_0: track 1.57 -> 13.0 mm
- net +22.2V_LOGIC_POWER_SENSOR_OUT: track 19.0 -> 8.41 mm
- net Net-(D2-A): track 10.3 -> 1.48 mm
- net BUFF_E_STOP_STATUS: track 40.8 -> 33.2 mm
- net +14.4V_DRIVE_BATT: track 0.00 -> 7.37 mm, vias 0 -> 12
- net Net-(U7-EN/UV): track 5.97 -> 1.05 mm
- net +20V_JETSON_VCC: track 4.37 -> 0.00 mm
- net Net-(U6-INTVCC): track 4.00 -> 0.00 mm
- net Net-(U8-RT): track 3.97 -> 0.00 mm
- net Net-(U4-EN): track 4.70 -> 1.06 mm
- net Net-(U8-EN/UV): track 4.55 -> 1.07 mm
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- added copper zone on F.Cu, net +14.4V_DRIVE1
- added copper zone on F.Cu, net +14.4V_DRIVE1_SENSOR_OUT
- added copper zone on F.Cu, net +14.4V_DRIVE2
- added copper zone on F.Cu, net +14.4V_DRIVE2_SENSOR_OUT
- added copper zone on F.Cu, net +14.4V_DRIVE3
- added copper zone on F.Cu, net +14.4V_DRIVE3_SENSOR_OUT
- added copper zone on F.Cu, net +14.4V_DRIVE4
- added copper zone on F.Cu, net +14.4V_DRIVE4_SENSOR_OUT
- added copper zone on F.Cu, net +14.4V_DRIVE5
- added copper zone on F.Cu, net +14.4V_DRIVE5_SENSOR_OUT
- added copper zone on F.Cu, net +14.4V_DRIVE6
- added copper zone on F.Cu, net +14.4V_DRIVE6_SENSOR_OUT
- added copper zone on F.Cu, net +14.4V_DRIVE_BATT
- added copper zone on F.Cu, net Net-(Q1-G)
- added copper zone on F.Cu, net Net-(Q2-G)
- added copper zone on F.Cu, net Net-(Q3-G)
- added copper zone on F.Cu, net Net-(Q4-G)
- added copper zone on F.Cu, net Net-(Q5-G)
- added copper zone on F.Cu, net Net-(Q6-G)
Other:
- board outline added: 240 x 85 mm

Commit message: Stuff
Parts:
- C2, C72: moved to F.Cu
- R47, R48, R49, R50, R51, R52, R53, R54, R55, R56, R59, R60, U13, U14: moved to B.Cu
- moved H3 236.8 mm to (32.2, 46.7)
- moved H1 222.6 mm to (255.6, 46.8)
- moved R47 79.8 mm to (147.4, 86.0)
- moved R55 79.8 mm to (147.4, 88.0)
- moved H2 73.9 mm to (255.9, 118.8)
- moved U13 72.5 mm to (143.7, 87.0)
- moved R59 72.3 mm to (143.6, 84.9), turned to 180 degrees
- moved R51 72.1 mm to (143.5, 89.1), turned to 0 degrees
- moved R49 65.2 mm to (140.0, 86.0)
- moved R53 65.2 mm to (140.0, 88.0)
- moved R48 62.8 mm to (147.5, 80.7)
- moved R56 62.8 mm to (147.5, 82.7)
- moved U14 55.3 mm to (143.7, 81.7)
- moved R60 55.1 mm to (143.6, 79.6), turned to 180 degrees
- moved R52 55.1 mm to (143.6, 83.8), turned to 0 degrees
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Connections:
- H1 pad 1: CHA_GND -> GND
- H2 pad 1: CHA_GND -> GND
- H3 pad 1: CHA_GND -> GND
- H4 pad 1: CHA_GND -> GND
Routing:
- net BUFF_SDA_0: track 1.59 -> 328.2 mm, vias 0 -> 10
- net BUFF_SDA_1: track 1.67 -> 92.2 mm, vias 0 -> 2
- net BUFF_SCL_0: track 13.0 -> 100.9 mm, vias 0 -> 4
- net BUFF_SCL_1: track 1.61 -> 83.4 mm, vias 0 -> 2
- net +3.3V_RP2350_VCC: track 164.4 -> 222.6 mm, vias 7 -> 9
- net BUFF_E_STOP_STATUS: track 33.2 -> 89.4 mm
- net /RP2350A/GPIO17: track 0.00 -> 31.2 mm, vias 0 -> 1
- net /RP2350A/GPIO19: track 0.00 -> 30.6 mm
- net /RP2350A/GPIO13: track 0.00 -> 30.3 mm
- net /RP2350A/GPIO22: track 0.00 -> 30.0 mm, vias 0 -> 1
- net /RP2350A/GPIO15: track 0.00 -> 29.8 mm
- net /RP2350A/GPIO16: track 0.00 -> 29.1 mm, vias 0 -> 1
- net /RP2350A/GPIO21: track 0.00 -> 28.9 mm, vias 0 -> 1
- net /RP2350A/GPIO18: track 0.00 -> 28.6 mm, vias 0 -> 1
- net /RP2350A/GPIO14: track 0.00 -> 27.7 mm
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- added copper zone on F.Cu, net +22.2V_LOGIC
Other:
- board size 240 x 85 mm -> 237.7 x 86.1 mm

Commit message: More Layout :)
Parts:
- moved C67 84.2 mm to (134.0, 149.1)
- moved C69 84.2 mm to (138.2, 149.1)
- moved C71 84.2 mm to (142.5, 149.1)
- moved R100 84.2 mm to (138.8, 156.3)
- moved R101 84.2 mm to (140.8, 156.3)
- moved R92 84.2 mm to (132.8, 153.4)
- moved R93 84.2 mm to (134.8, 153.4)
- moved R94 84.2 mm to (136.8, 153.4)
- moved R95 84.2 mm to (138.8, 153.4)
- moved R96 84.2 mm to (140.8, 153.4)
- moved R97 84.2 mm to (132.8, 156.3)
- moved R98 84.2 mm to (134.8, 156.3)
- moved R99 84.2 mm to (136.8, 156.3)
- moved U36 84.2 mm to (148.1, 148.7)
- moved C60 84.2 mm to (133.1, 144.3)
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Routing:
- net BUFF_SDA_0: track 328.2 -> 45.6 mm, vias 10 -> 7
- net BUFF_SDA_1: track 92.2 -> 1.67 mm
- net BUFF_SCL_0: track 100.9 -> 15.8 mm
- net BUFF_SCL_1: track 83.4 -> 1.61 mm
- net +14.4V_DRIVE_BATT: vias 13 -> 10
- net GND: vias 198 -> 195
- net /Subsystem Power Control/GATE_DRIVE3: vias 0 -> 1
- net /Subsystem Power Control/GATE_DRIVE2: vias 0 -> 1
- net /Subsystem Power Control/GATE_DRIVE1: vias 0 -> 1
Other:
- board outline removed

Commit message: More layout!
Parts:
- moved R97 81.6 mm to (173.2, 85.4), turned to 0 degrees
- moved R95 71.8 mm to (170.9, 89.2)
- moved R100 71.3 mm to (171.7, 93.0)
- moved R94 69.4 mm to (147.3, 84.8), turned to 0 degrees
- moved R96 69.1 mm to (170.9, 91.2)
- moved C61 67.8 mm to (170.9, 86.4)
- moved R101 66.8 mm to (158.0, 91.7), turned to 180 degrees
- moved R92 66.2 mm to (145.0, 88.3)
- moved R98 64.7 mm to (145.5, 92.5)
- moved R99 64.6 mm to (131.8, 91.9), turned to 180 degrees
- moved R93 63.9 mm to (145.0, 90.3)
- moved U36 60.7 mm to (153.4, 88.2), turned to 0 degrees
- moved C64 60.0 mm to (174.0, 92.8), turned to 180 degrees
- moved C60 59.9 mm to (145.0, 85.6)
- moved C65 52.6 mm to (158.2, 93.2), turned to 180 degrees
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Routing:
- net Net-(U31-TS): track 0.00 -> 17.7 mm, vias 0 -> 1
- net Net-(U32-TS): track 0.00 -> 16.6 mm, vias 0 -> 1
- net Net-(U32-OVLO): track 0.00 -> 4.39 mm
- net Net-(U31-OVLO): track 0.00 -> 4.07 mm
- net Net-(U31-TGUP): track 0.00 -> 3.07 mm
- net Net-(U32-TGUP): track 0.00 -> 2.97 mm
- net Net-(U31-BST): track 0.00 -> 2.72 mm
- net Net-(U32-BST): track 0.00 -> 2.21 mm
- net Net-(Q7-G): track 0.00 -> 1.85 mm
- net Net-(Q8-G): track 0.00 -> 1.75 mm
- net /RP2350A/SWD: track 9.32 -> 11.1 mm
- net /RP2350A/SWCLK: track 11.8 -> 13.4 mm
- net Net-(U31-VCCUV): track 0.00 -> 1.51 mm
- net Net-(U32-VCCUV): track 0.00 -> 1.43 mm
- net /RP2350A/RUN: track 6.23 -> 7.27 mm
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- added copper zone on In2.Cu, net GND
