File: BILLEE_Rover_Control_Module_V1/BILLEE_Rover_Control_Module_V1.kicad_pcb (KiCad board)
At the start: 4 copper layers, 271 parts, among them CN1 XT90PW-M.G.Y, CN10 XT60PW-M, CN11 XT60PW-M, CN12 XT60PW-M, CN13 XT60PW-M, CN14 XT60PW-M, CN15 XT60PW-M, CN16 XT60PW-M, CN17 XT60PW-M, CN18 XT60PW-M, CN2 XT60PW-M, CN3 XT60PW-M, CN4 XT60PW-M, CN5 XT60PW-M, CN6 DF11-18DP-2DSA, CN7 XT90PW-M.G.Y, CN8 XT90PW-M.G.Y, CN9 XT90PW-M.G.Y, J1 2.54mm Header, Q1 IPT007N06N, Q2 IPT007N06N, Q3 IPT007N06N, Q4 IPT007N06N, Q5 IPT007N06N, Q6 IPT007N06N, Q7 IPT007N06N, Q8 IPT007N06N, SW1 33uH, SW2 KMR2, SW3 RESET SW, U1 INA780BIDEKR, U10 RP2350A_C42411118, U11 ABM8-272-T3_C20625731, U12 W25Q128JVSIQTR, U13 TCA4307DGKR, U14 TCA4307DGKR, U15 TXS0108EPWR, U16 ESTOP, U17 SN74LVC08APWR, U18 SN74LVC08APWR, U19 LTC7001IMSE#PBF, U2 MCP9808T-E/MS, U20 LTC7001IMSE#PBF, U21 LTC7001IMSE#PBF, U22 LTC7001IMSE#PBF, U23 LTC7001IMSE#PBF, U24 LTC7001IMSE#PBF, U25 INA780BIDEKR, U26 INA780BIDEKR, U27 INA780BIDEKR, U28 INA780BIDEKR, U29 INA780BIDEKR, U3 TPS1HA08BQPWPRQ1, U30 INA780BIDEKR, U31 LTC7001IMSE#PBF, U32 LTC7001IMSE#PBF, U33 INA780BIDEKR, U34 INA780BIDEKR, U35 MCP9808T-E/MS, U36 MCP9808T-E/MS, U4 TPS1HA08BQPWPRQ1, U5 TPS1HA08BQPWPRQ1, U6 LT8612EUDE#TRPBF, U7 LT8612EUDE#TRPBF, U8 LT8612EUDE#TRPBF, U9 10uH

Commit message: Stuffffff
Routing:
- net +14.4V_DRIVE_BATT: track 18.8 -> 91.2 mm, vias 10 -> 12
- net +12V_AUX_VCC: track 0.00 -> 43.6 mm, vias 0 -> 3
- net Net-(U20-TS): track 2.24 -> 8.57 mm
- net Net-(U24-TS): track 2.24 -> 8.57 mm
- net Net-(U22-TS): track 2.24 -> 8.57 mm
- net Net-(U21-TS): track 2.24 -> 8.57 mm
- net Net-(U23-TS): track 2.24 -> 8.57 mm
- net Net-(U19-TS): track 2.24 -> 8.57 mm
- net PI_SDA_1: vias 2 -> 1
- net PI_SDA_0: vias 2 -> 1
- net PI_SCL_1: vias 2 -> 1
- net PI_SCL_0: vias 2 -> 1

Commit message: Fixed board outline
Parts:
- moved H1 1.56 mm to (255.6, 45.2)
- moved H3 1.51 mm to (32.1, 45.2)
- moved H4 1.09 mm to (32.1, 119.8)
- moved H2 1.03 mm to (255.6, 119.8)
Other:
- board outline added: 237.5 x 88.6 mm
Changed lines of the file:
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@@
 	(footprint "MountingHole:MountingHole_4.3mm_M4_Pad_Via"
 		(layer "F.Cu")
-		(at 32.2 46.725)
+		(at 32.14 45.22)
 		(descr "Mounting Hole 4.3mm, M4, generated by kicad-footprint-generator mountinghole.py")
 		(tags "mountinghole M4")
@@
 	(footprint "MountingHole:MountingHole_4.3mm_M4_Pad_Via"
 		(layer "F.Cu")
-		(at 255.60407 46.78009)
+		(at 255.59 45.22)
 		(descr "Mounting Hole 4.3mm, M4, generated by kicad-footprint-generator mountinghole.py")
 		(tags "mountinghole M4")
@@
 	(footprint "MountingHole:MountingHole_4.3mm_M4_Pad_Via"
 		(layer "F.Cu")
-		(at 32.519581 118.819581)
+		(at 32.120419 119.830429)
 		(descr "Mounting Hole 4.3mm, M4, generated by kicad-footprint-generator mountinghole.py")
 		(tags "mountinghole M4")
@@
 	(footprint "MountingHole:MountingHole_4.3mm_M4_Pad_Via"
 		(layer "F.Cu")
-		(at 255.90909 118.84616)
+		(at 255.57409 119.81617)
 		(descr "Mounting Hole 4.3mm, M4, generated by kicad-footprint-generator mountinghole.py")
 		(tags "mountinghole M4")
@@
 	)
 	(gr_line
-		(start 25.539162 118.839162)
-		(end 32.539162 118.839162)
+		(start 25.13 45.22)
+		(end 25.13 119.85001)
 		(stroke
 			(width 0.05)
 			(type solid)
 		)
-		(layer "Dwgs.User")
+		(layer "Edge.Cuts")
 	)
-	(gr_line
-		(start 32.2 40)
-		(end 32.2 47)
+	(gr_arc
+		(start 25.13 45.22)
+		(mid 27.180247 40.260247)
+		(end 32.14 38.21)
 		(stroke
 			(width 0.05)
-			(type solid)
+			(type default)
 		)
-		(layer "Dwgs.User")
+		(layer "Edge.Cuts")
 	)
-	(gr_line
-		(start 32.2 47)
-		(end 25.2 47)
+	(gr_arc
+		(start 32.12 126.830007)
+		(mid 27.180859 124.786219)
+		(end 25.13 119.85001)
 		(stroke
 			(width 0.05)
-			(type solid)
+			(type default)
 		)
-		(layer "Dwgs.User")
+		(layer "Edge.Cuts")
 	)
 	(gr_line
-		(start 32.539162 118.839162)
-		(end 32.539162 125.839162)
+		(start 32.12 126.830007)
+		(end 255.580006 126.836982)
 		(stroke
 			(width 0.05)
 			(type solid)
 		)
-		(layer "Dwgs.User")
+		(layer "Edge.Cuts")
 	)
 	(gr_line
-		(start 255.585838 46.760838)
-		(end 255.585838 39.760838)
+		(start 32.14 38.21)
+		(end 255.58 38.21)
 		(stroke
 			(width 0.05)
 			(type solid)
 		)
-		(layer "Dwgs.User")
+		(layer "Edge.Cuts")
 	)
-	(gr_line
-		(start 255.925 118.6)
-		(end 262.925 118.6)
+	(gr_arc
+		(start 255.58 38.21)
+		(mid 260.543287 40.259642)
+		(end 262.600007 45.22)
 		(stroke
 			(width 0.05)
-			(type solid)
+			(type default)
 		)
-		(layer "Dwgs.User")
+		(layer "Edge.Cuts")
 	)
-	(gr_line
-		(start 255.925 125.6)
-		(end 255.925 118.6)
+	(gr_arc
+		(start 262.59 119.57001)
+		(mid 260.62667 124.690647)
+		(end 255.580006 126.836982)
 		(stroke
 			(width 0.05)
-			(type solid)
+			(type default)
 		)
-		(layer "Dwgs.User")
+		(layer "Edge.Cuts")
 	)
 	(gr_line
-		(start 262.585838 46.760838)
-		(end 255.585838 46.760838)
+		(start 262.600007 45.22)
+		(end 262.59 119.57001)
 		(stroke
 			(width 0.05)
 			(type solid)
 		)
-		(layer "Dwgs.User")
+		(layer "Edge.Cuts")
 	)
 	(gr_text "C2150178"
@@
 	)
 	(via
-		(at 196 61.4)
+		(at 195.9546 60.922)
 		(size 0.3)
 		(drill 0.15)
@@
 	)
 	(via
-		(at 237.3 61.5)
+		(at 237.1976 60.9676)
 		(size 0.3)
 		(drill 0.15)
@@
 		)
 		(min_thickness 0.25)
-		(fill
+		(fill yes
 			(thermal_gap 0.5)
 			(thermal_bridge_width 0.5)

Commit message: More layout :tired_face:
Routing:
- net BUFF_SDA_0: track 45.6 -> 291.6 mm, vias 6 -> 10
- net +12V_AUX_VCC: track 43.6 -> 263.2 mm, vias 3 -> 8
- net BUFF_SCL_0: track 15.8 -> 190.3 mm, vias 4 -> 12
- net PI_SCL_0: track 1.55 -> 45.2 mm, vias 1 -> 2
- net +14.4V_ARM_BATT: track 0.00 -> 8.24 mm
- net +3.3V_RP2350_VCC: track 222.6 -> 219.3 mm
- net PI_SCL_1: track 1.52 -> 3.35 mm, vias 1 -> 2
- net PI_SDA_0: track 1.56 -> 3.30 mm, vias 1 -> 2
- net Net-(C65-Pad2): track 0.00 -> 1.54 mm
- net PI_SDA_1: track 1.67 -> 3.17 mm, vias 1 -> 2
- net Net-(C63-Pad2): track 0.00 -> 1.38 mm
- net Net-(U34-IN–): track 0.00 -> 0.95 mm
- net Net-(U34-IN+): track 0.00 -> 0.75 mm
- net GND: vias 214 -> 219
- added copper zone on F.Cu, net +14.4V_SCIENCE_BATT
- added copper zone on B.Cu, net GND
- added copper zone on F.Cu, net GND
- added copper zone on In1.Cu, net GND
- added copper zone on F.Cu, net Net-(Q7-G)
- added copper zone on F.Cu, net Net-(Q8-G)

Commit message: Resatarted Layout for something a little bit cleaner.
Parts:
- removed TP1, TP3: TestPoint, TestPoint:TestPoint_THTPad_2.0x2.0mm_Drill1.0mm
- U15: moved to F.Cu
- U17, U18: moved to B.Cu
- moved U16 29.0 mm to (50.0, 52.5)
- moved R61 28.5 mm to (55.0, 60.5), turned to 90 degrees
- moved CN7 20.0 mm to (175.3, 62.3)
- moved CN9 19.1 mm to (139.3, 62.3)
- moved CN8 18.4 mm to (103.3, 62.3)
- moved CN1 17.1 mm to (67.3, 62.3)
- moved U2 14.1 mm to (57.4, 89.2), turned to 90 degrees
- moved C24 10.7 mm to (107.7, 96.0), turned to 90 degrees
- moved U35 10.6 mm to (214.4, 73.4), turned to -90 degrees
- moved C72 10.4 mm to (54.1, 86.6), turned to 0 degrees
- moved R39 9.64 mm to (87.2, 110.5)
- moved U1 9.60 mm to (66.5, 80.0), turned to 0 degrees
- moved C4 9.07 mm to (53.0, 89.0), turned to 90 degrees
- moved U17 8.71 mm to (103.9, 109.8)
- moved D1 8.52 mm to (60.5, 82.5)
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Routing:
- net BUFF_SDA_0: track 291.6 -> 0.00 mm, vias 10 -> 0
- net +12V_AUX_VCC: track 263.2 -> 0.00 mm, vias 8 -> 0
- net +3.3V_RP2350_VCC: track 219.3 -> 0.00 mm, vias 9 -> 0
- net BUFF_SCL_0: track 190.3 -> 2.92 mm, vias 12 -> 0
- net +14.4V_DRIVE_BATT: track 91.2 -> 0.00 mm, vias 12 -> 0
- net BUFF_E_STOP_STATUS: track 89.4 -> 7.07 mm, vias 3 -> 0
- net +14.4V_SCIENCE_BATT: track 0.00 -> 49.4 mm
- net PI_SCL_0: track 45.2 -> 0.00 mm, vias 2 -> 0
- net +14.4V_ARM_BATT: track 8.24 -> 47.5 mm
- net GND: track 34.0 -> 0.00 mm, vias 219 -> 227
- net /RP2350A/GPIO17: track 31.2 -> 0.00 mm, vias 1 -> 0
- net /RP2350A/GPIO19: track 30.3 -> 0.00 mm, vias 1 -> 0
- net /RP2350A/GPIO13: track 30.3 -> 0.00 mm, vias 1 -> 0
- net /RP2350A/GPIO22: track 30.0 -> 0.00 mm, vias 1 -> 0
- net +14.4V_SCIENCE_SENSOR_OUT: track 0.00 -> 30.0 mm
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- added copper zone on F.Cu, net +14.4V_ARM_SENSOR_OUT
- removed copper zone on F.Cu, net +14.4V_DRIVE1
- removed copper zone on F.Cu, net +14.4V_DRIVE1_SENSOR_OUT
- removed copper zone on F.Cu, net +14.4V_DRIVE2
- removed copper zone on F.Cu, net +14.4V_DRIVE2_SENSOR_OUT
- removed copper zone on F.Cu, net +14.4V_DRIVE3
- removed copper zone on F.Cu, net +14.4V_DRIVE3_SENSOR_OUT
- removed copper zone on F.Cu, net +14.4V_DRIVE4
- removed copper zone on F.Cu, net +14.4V_DRIVE4_SENSOR_OUT
- removed copper zone on F.Cu, net +14.4V_DRIVE5
- removed copper zone on F.Cu, net +14.4V_DRIVE5_SENSOR_OUT
- removed copper zone on F.Cu, net +14.4V_DRIVE6
- removed copper zone on F.Cu, net +14.4V_DRIVE6_SENSOR_OUT
- removed copper zone on F.Cu, net +14.4V_SCIENCE_BATT
- removed copper zone on F.Cu, net +22.2V_LOGIC
- removed copper zone on In2.Cu, net GND
- removed copper zone on F.Cu, net Net-(Q1-G)
- removed copper zone on F.Cu, net Net-(Q2-G)
- removed copper zone on F.Cu, net Net-(Q3-G)
- removed copper zone on F.Cu, net Net-(Q4-G)
- removed copper zone on F.Cu, net Net-(Q5-G)
- removed copper zone on F.Cu, net Net-(Q6-G)
- removed copper zone on F.Cu, net Net-(Q7-G)
- removed copper zone on F.Cu, net Net-(Q8-G)
- removed copper zone on F.Cu, net Net-(U5-VOUT)
- removed copper zone on F.Cu, net Net-(U6-FB)
- removed copper zone on F.Cu, net Net-(U6-SW)
- removed copper zone on F.Cu, net Net-(U7-FB)
- removed copper zone on F.Cu, net Net-(U7-SW)
- removed copper zone on F.Cu, net Net-(U8-FB)
- removed copper zone on F.Cu, net Net-(U8-SW)
Other:
- board size 237.5 x 88.6 mm -> 240 x 90.5 mm

Commit message: Routing continued
Parts:
- U15: moved to B.Cu
- U17, U18: moved to F.Cu
- moved R55 15.1 mm to (125.3, 72.9), turned to 0 degrees
- moved R51 13.3 mm to (126.4, 76.8), turned to 90 degrees
- moved R47 13.2 mm to (123.3, 72.9), turned to 180 degrees
- moved R56 11.2 mm to (120.0, 72.8), turned to 0 degrees
- moved D3 11.2 mm to (102.4, 81.0)
- moved R53 10.7 mm to (125.3, 80.3), turned to 0 degrees
- moved R48 10.7 mm to (118.0, 72.8), turned to 180 degrees
- moved U13 10.7 mm to (124.3, 76.6), turned to 180 degrees
- moved R59 8.24 mm to (122.2, 76.7), turned to -90 degrees
- moved R49 7.92 mm to (123.3, 80.3), turned to 180 degrees
- moved R60 6.83 mm to (117.0, 74.4), turned to 90 degrees
- moved U17 6.22 mm to (97.7, 109.2)
- moved U18 5.96 mm to (97.7, 104.0), turned to -90 degrees
- moved U14 5.66 mm to (119.0, 76.6), turned to 180 degrees
- moved R52 4.98 mm to (121.0, 78.8), turned to -90 degrees
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Routing:
- net /Subsystem Power Control/GATE_DRIVE3: track 0.00 -> 179.0 mm, vias 0 -> 2
- net /Subsystem Power Control/GATE_DRIVE4: track 0.00 -> 153.3 mm, vias 0 -> 2
- net /Subsystem Power Control/GATE_DRIVE2: track 0.00 -> 135.7 mm, vias 0 -> 2
- net /Subsystem Power Control/GATE_DRIVE5: track 0.00 -> 127.8 mm, vias 0 -> 2
- net /Subsystem Power Control/GATE_DRIVE1: track 0.00 -> 119.7 mm, vias 0 -> 2
- net +12V_AUX_VCC: track 0.00 -> 113.4 mm, vias 0 -> 8
- net /Subsystem Power Control/GATE_DRIVE6: track 0.00 -> 109.9 mm, vias 0 -> 2
- net BUFF_E_STOP_STATUS: track 7.07 -> 115.8 mm, vias 0 -> 1
- net /Subsystem Power Control/GATE_ARM: track 0.00 -> 84.0 mm, vias 0 -> 2
- net /Subsystem Power Control/GATE_SCIENCE: track 0.00 -> 53.9 mm, vias 0 -> 2
- net /RP2350A/GPIO13: track 0.00 -> 37.4 mm, vias 0 -> 1
- net /RP2350A/GPIO15: track 0.00 -> 36.9 mm, vias 0 -> 1
- net /RP2350A/GPIO14: track 0.00 -> 34.7 mm, vias 0 -> 1
- net /RP2350A/GPIO17: track 0.00 -> 30.5 mm, vias 0 -> 1
- net /RP2350A/GPIO19: track 0.00 -> 30.3 mm, vias 0 -> 1
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- added copper zone on F.Cu, net +14.4V_SCIENCE_SENSOR_OUT
- added copper zone on F.Cu, net Net-(U5-VOUT)
- added copper zone on F.Cu, net Net-(U7-SW)
- added copper zone on F.Cu, net Net-(U8-SW)
