File: BILLEE_Rover_Control_Module_V1/BILLEE_Rover_Control_Module_V1.kicad_pcb (KiCad board)
At the start: 4 copper layers, 240 x 90.5 mm, 276 parts, among them CN1 XT90PW-M.G.Y, CN10 XT60PW-M, CN11 XT60PW-M, CN12 XT60PW-M, CN13 XT60PW-M, CN14 XT60PW-M, CN15 XT60PW-M, CN16 XT60PW-M, CN17 XT60PW-M, CN18 XT60PW-M, CN2 XT60PW-M, CN3 XT60PW-M, CN4 XT60PW-M, CN5 XT60PW-M, CN6 DF11-18DP-2DSA, CN7 XT90PW-M.G.Y, CN8 XT90PW-M.G.Y, CN9 XT90PW-M.G.Y, J1 2.54mm Header, Q1 IPT007N06N, Q2 IPT007N06N, Q3 IPT007N06N, Q4 IPT007N06N, Q5 IPT007N06N, Q6 IPT007N06N, Q7 IPT007N06N, Q8 IPT007N06N, SW1 33uH, SW2 KMR2, SW3 RESET SW, U1 INA780BIDEKR, U10 RP2350A_C42411118, U11 ABM8-272-T3_C20625731, U12 W25Q128JVSIQTR, U13 TCA4307DGKR, U14 TCA4307DGKR, U15 TXS0108EPWR, U16 ESTOP, U17 SN74LVC08APWR, U18 SN74LVC08APWR, U19 LTC7001IMSE#PBF, U2 MCP9808T-E/MS, U20 LTC7001IMSE#PBF, U21 LTC7001IMSE#PBF, U22 LTC7001IMSE#PBF, U23 LTC7001IMSE#PBF, U24 LTC7001IMSE#PBF, U25 INA780BIDEKR, U26 INA780BIDEKR, U27 INA780BIDEKR, U28 INA780BIDEKR, U29 INA780BIDEKR, U3 TPS1HA08BQPWPRQ1, U30 INA780BIDEKR, U31 LTC7001IMSE#PBF, U32 LTC7001IMSE#PBF, U33 INA780BIDEKR, U34 INA780BIDEKR, U35 MCP9808T-E/MS, U36 MCP9808T-E/MS, U4 TPS1HA08BQPWPRQ1, U5 TPS1HA08BQPWPRQ1, U6 LT8612EUDE#TRPBF, U7 LT8612EUDE#TRPBF, U8 LT8612EUDE#TRPBF, U9 10uH

Commit message: Applied Jason Suarez Feeback
Updated Inductor value from 1.8u to 8.2u for correct ringing match. Regenerated Gerbers and BOM
Parts:
- L1: value 1.8u -> 8.2u
Changed lines of the file:
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@@
 		(sheetname "/RP2350A/")
 		(sheetfile "mcurp2350.kicad_sch")
+		(units
+			(unit
+				(name "A")
+				(pins "9" "3" "13" "14" "12" "1" "2" "11" "4" "10" "7" "5" "6" "8")
+			)
+		)
 		(attr smd)
 		(duplicate_pad_numbers_are_jumpers no)
@@
 			)
 		)
-		(property "Value" "1.8u"
+		(property "Value" "8.2u"
 			(at 0 4 0)
 			(layer "F.Fab")
@@
 			)
 		)
-		(property "Datasheet" "https://lcsc.com/product-detail/Inductors-SMD_TDK_NLV32T-1R8J-PF_NLV32T-1R8J-PF_C41039.html"
+		(property "Datasheet" "https://www.lcsc.com/datasheet/C318062.pdf?spm=wm.sxq.inf.ggs&utm_source=chatgpt.com&lcsc_vid=FVENUldeFQQKA1xfRQAPUVZTRQcKAgFSE1ZZV1wCFQcxVlNeQFRbUFBXRFFdUDsOAxUeFF5JWAIGBhABBxVABAsLWA%3D%3D"
 			(at 0 0 0)
 			(layer "F.Fab")
@@
 			)
 		)
-		(property "LCSC Part" "C41039"
+		(property "LCSC Part" "C318062"
 			(at 0 0 0)
 			(layer "F.Fab")
@@
 			)
 		)
-		(property "Manufacturer" "TDK"
+		(property "Manufacturer" ""
 			(at 0 0 180)
 			(unlocked yes)
@@
 			)
 		)
-		(property "MPN" "NLV32T-1R8J-PF"
+		(property "MPN" "FHW1210HC8R2JGT"
 			(at 0 0 180)
 			(unlocked yes)

Commit message: Updated some values, updated their sims. Ready for a Claude Pass.
Parts:
- C17: value 10p -> 4.7p
- C20, C23: value 10u -> 22u
Changed lines of the file:
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@@
 	(title_block
 		(title "Perserverance")
-		(date "2026-08-22")
+		(date "2026-08-26")
 		(rev "V1")
 		(company "Bronco STAR")
-		(comment 1 "With love to all. Thank you for this opportunity to make this")
+		(comment 1 "-Luca")
+		(comment 2 "Thank you for trusting me and providing the opportunity to make this")
 	)
 	(layers
@@
 			)
 		)
-		(property "Value" "10u"
+		(property "Value" "22u"
 			(at 0 1 0)
 			(layer "F.Fab")
@@
 			)
 		)
+		(property "LCSC" "C3845593"
+			(at 0 0 0)
+			(layer "F.SilkS")
+			(hide yes)
+			(effects
+				(font
+					(size 1.27 1.27)
+					(thickness 0.15)
+				)
+			)
+		)
 		(property ki_fp_filters "C_*")
 		(sheetname "/Logic Subsystem/")
@@
 			)
 		)
-		(property "Value" "10p"
+		(property "Value" "4.7p"
 			(at 0 1.43 0)
 			(layer "F.Fab")
@@
 			)
 		)
-		(property "Value" "10u"
+		(property "Value" "22u"
 			(at 0 1 0)
 			(layer "F.Fab")
@@
 					(thickness 0.15)
 				)
+			)
+		)
+		(property "LCSC" "C3845593"
+			(at 0 0 0)
+			(layer "F.SilkS")
+			(hide yes)
+			(effects
+				(font
+					(size 1.27 1.27)
+					(thickness 0.15)
+				)

Commit message: Updated with Claude Notes. Checking again.
Parts:
- C20, C23: footprint Capacitor_SMD:C_01005_0402Metric -> Capacitor_SMD:C_0402_1005Metric
- moved R32 0.86 mm to (85.1, 94.0)
- moved R35 0.86 mm to (85.1, 92.9)
- moved C23 0.64 mm to (83.0, 94.0)
- moved C20 0.45 mm to (83.0, 93.0)
Routing:
- net +14.4V_SCIENCE_SENSOR_OUT: track 25.3 -> 31.0 mm
- net +14.4V_ARM_SENSOR_OUT: track 31.6 -> 32.8 mm
