File: BILLEE_Rover_Control_Module_V1/mcurp2350.kicad_sch (KiCad schematic)
At the start: 54 parts, among them CN14 DF11-18DP-2DSA, J1 2.54mm Header, SW2 KMR2, SW3 RESET SW, U15 W25Q128JVSIQTR, U17 ABM8-272-T3_C20625731, U18 RP2350A_C42411118, U19 TXS0108EPWR, U21 TCA4307DGKR, U22 TCA4307DGKR

Commit message: Biggus Goodies
Parts:
- D1: footprint (none) -> Diode_SMD:D_0805_2012Metric; LCSC Part (none) -> C84260
- R12, R13, R14, R15, R16, R17, R18, R19, R20, R21, R22, R23: footprint (none) -> Resistor_SMD:R_0402_1005Metric
- R25: value 2k -> 330; footprint (none) -> Resistor_SMD:R_0402_1005Metric
Changed lines of the file:
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@@
 			)
 		)
-		(property "Footprint" ""
+		(property "Footprint" "Resistor_SMD:R_0402_1005Metric"
 			(at 312.674 129.286 90)
 			(hide yes)
@@
 			)
 		)
-		(property "Footprint" ""
+		(property "Footprint" "Resistor_SMD:R_0402_1005Metric"
 			(at 362.204 129.286 90)
 			(hide yes)
@@
 			)
 		)
-		(property "Footprint" ""
+		(property "Footprint" "Resistor_SMD:R_0402_1005Metric"
 			(at 320.294 129.286 90)
 			(hide yes)
@@
 			)
 		)
-		(property "Footprint" ""
+		(property "Footprint" "Diode_SMD:D_0805_2012Metric"
 			(at 224.79 43.18 0)
 			(hide yes)
@@
 			)
 		)
-		(property "Datasheet" ""
+		(property "Datasheet" "https://www.lcsc.com/datasheet/C84260.pdf?spm=wm.sxq.inf.ggs___wm.fly.bg.0.xh&lcsc_vid=TlVbAVcAQABWBFIHTlJdAQJeElcNAVNeFlQKBFBfQVIxVlNeQVBZVVNVQlFaVTsOAxUeFF5JWBYZEEoKFBINSQcJGk4%3D"
 			(at 224.79 43.18 0)
 			(hide yes)
@@
 			)
 		)
+		(property "LCSC Part" "C84260"
+			(at 224.79 43.18 90)
+			(hide yes)
+			(show_name no)
+			(do_not_autoplace no)
+			(effects
+				(font
+					(size 1.27 1.27)
+				)
+			)
+		)
 		(pin "2"
 		)
@@
 			)
 		)
-		(property "Value" "2k"
+		(property "Value" "330"
 			(at 226.568 37.084 0)
 			(show_name no)
@@
 			)
 		)
-		(property "Footprint" ""
+		(property "Footprint" "Resistor_SMD:R_0402_1005Metric"
 			(at 225.806 35.814 90)
 			(hide yes)
@@
 			)
 		)
-		(property "Footprint" ""
+		(property "Footprint" "Resistor_SMD:R_0402_1005Metric"
 			(at 371.094 94.996 90)
 			(hide yes)
@@
 			)
 		)
-		(property "Footprint" ""
+		(property "Footprint" "Resistor_SMD:R_0402_1005Metric"
 			(at 379.984 94.996 90)
 			(hide yes)
@@
 			)
 		)
-		(property "Footprint" ""
+		(property "Footprint" "Resistor_SMD:R_0402_1005Metric"
 			(at 327.914 94.996 90)
 			(hide yes)
@@
 			)
 		)
-		(property "Footprint" ""
+		(property "Footprint" "Resistor_SMD:R_0402_1005Metric"
 			(at 362.204 94.996 90)
 			(hide yes)
@@
 			)
 		)
-		(property "Footprint" ""
+		(property "Footprint" "Resistor_SMD:R_0402_1005Metric"
 			(at 371.094 129.286 90)
 			(hide yes)
@@
 			)
 		)
-		(property "Footprint" ""
+		(property "Footprint" "Resistor_SMD:R_0402_1005Metric"
 			(at 320.294 94.996 90)
 			(hide yes)
@@
 			)
 		)
-		(property "Footprint" ""
+		(property "Footprint" "Resistor_SMD:R_0402_1005Metric"
 			(at 327.914 129.286 90)
 			(hide yes)
@@
 			)
 		)
-		(property "Footprint" ""
+		(property "Footprint" "Resistor_SMD:R_0402_1005Metric"
 			(at 379.984 129.286 90)
 			(hide yes)
@@
 			)
 		)
-		(property "Footprint" ""
+		(property "Footprint" "Resistor_SMD:R_0402_1005Metric"
 			(at 312.674 94.996 90)
 			(hide yes)

Commit message: Schematic Fixed in NO RCP yet
Parts:
- C65: footprint Capacitor_SMD:C_0402_1005Metric -> Capacitor_SMD:C_0603_1608Metric
Changed lines of the file:
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@@
 			)
 		)
-		(property "Footprint" "Capacitor_SMD:C_0402_1005Metric"
+		(property "Footprint" "Capacitor_SMD:C_0603_1608Metric"
 			(at 371.1448 160.02 0)
 			(hide yes)

Commit message: Updated footprint selection
Still missing the four inductors for the regulators, two of them can be poached from scales
Parts:
- C2, C3, C65: footprint Capacitor_SMD:C_0603_1608Metric -> Capacitor_SMD:C_0402_1005Metric
Changed lines of the file:
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@@
 			)
 		)
-		(property "Footprint" "Capacitor_SMD:C_0603_1608Metric"
+		(property "Footprint" "Capacitor_SMD:C_0402_1005Metric"
 			(at 32.7152 83.82 0)
 			(hide yes)
@@
 			)
 		)
-		(property "Footprint" "Capacitor_SMD:C_0603_1608Metric"
+		(property "Footprint" "Capacitor_SMD:C_0402_1005Metric"
 			(at 371.1448 160.02 0)
 			(hide yes)
@@
 			)
 		)
-		(property "Footprint" "Capacitor_SMD:C_0603_1608Metric"
+		(property "Footprint" "Capacitor_SMD:C_0402_1005Metric"
 			(at 44.1452 83.82 0)
 			(hide yes)

Commit message: Updated footprints. I think schematic is officially finished.
Parts:
- removed D1: PWR_LED, Diode_SMD:D_0805_2012Metric, symbol Device:LED
- removed L1: 3.3u, symbol Device:L
- added L4: 3.3u, PDB_LCSC:IND-SMD_L2.0-W1.6_AOTA-B201610S3R3-101-T, symbol PDB_LCSC_Libs:AOTA-B201610S3R3-101-T
- added LED1: FC-2012UGK-520D5, PDB_LCSC:LED0805-R-RD, symbol PDB_LCSC_Libs:FC-2012UGK-520D5
Connections:
- net +1V1: now also L4.2
- net GND: now also LED1.2 (K)
- net VREG_LX: now also L4.1
- net at R25.2: now also LED1.1 (A)

Commit message: Updated reference designators. Schematic Complete
Not including RCP for Drivetrain/Arm/Science
Parts:
- renumbered C2 to C25, C3 to C26, C42 to C27, C5 to C28, C43 to C29, C44 to C30, C6 to C31, C7 to C32, C8 to C33, C9 to C34, C10 to C35, C11 to C36, C12 to C37, C13 to C38, C14 to C39, C4 to C40, C65 to C41, CN14 to CN6, L4 to L2, R3 to R37, R5 to R38, R6 to R39, R7 to R40, R8 to R41, R25 to R42, R1 to R43, R2 to R44, R4 to R45, R11 to R46, R14 to R47, R18 to R48, R12 to R49, R19 to R50, R13 to R51, R20 to R52, R15 to R53, R21 to R54, R16 to R55, R22 to R56, R9 to R57, R10 to R58, R17 to R59, R23 to R60, U18 to U10, U17 to U11, U15 to U12, U21 to U13, U22 to U14, U19 to U15, USB2 to USB1

Commit message: More layout :tired_face:
Other:
- moved on the sheet: C38, C39, C41, R46, R47, R48, R49, R50, R51, R52, R53, R54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

Commit message: Updated with Claude Notes. Checking again.
Parts:
- R43: now not fitted
Changed lines of the file:
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@@
 		(in_pos_files yes)
 		(dnp no)
-		(fields_autoplaced yes)
 		(property "Reference" "U11"
 			(at 209.55 207.01 0)
@@
 		)
 		(property "Value" "ABM8-272-T3_C20625731"
-			(at 194.31 207.01 0)
-			(hide yes)
+			(at 203.962 199.898 90)
 			(show_name no)
 			(do_not_autoplace no)
@@
 		(on_board yes)
 		(in_pos_files yes)
-		(dnp no)
+		(dnp yes)
 		(property "Reference" "R43"
 			(at 252.73 33.528 90)
